File: MCU.kicad_sch (KiCad schematic)
At the start: 98 parts, among them IC1 MT2492, J1 FH34SRJ-8S-0.5SH_50_, J3 USB_C_Receptacle_USB2.0_16P, SW1 TS-1088-AR02016, SW2 TS-1088-AR02016, SW3 TS-1088-AR02016, U1 TEENSY 4.0, U2 ESP32-C3-MINI-1-H4X, U20 ATSAMD51J19A-A, U21 USBLC6-2SC6, U3 TLV75733PDBV, Y1 32.768kHz

Commit message: Made passives smaller from 0603 to 0402 because I will solder them with hot air gun anyway. Started positioning SAMD51 bypass caps.
Parts:
- removed C10: 100nF/50V, Capacitor_SMD:C_0603_1608Metric, symbol Device:C
- removed C11, C25, C27, C28, C8, C9: 47uF, Capacitor_SMD:C_1206_3216Metric, symbol Device:C
- removed C13: 2.2uF/25V, Capacitor_SMD:C_0603_1608Metric, symbol Device:C
- removed C14, C15, C29: 47uF/25V, Capacitor_SMD:C_1206_3216Metric, symbol Device:C
- removed C46: 100nF, Capacitor_SMD:C_0603_1608Metric, symbol Device:C
- added C47, C48: 100uF/25V, Capacitor_SMD:CP_Elec_6.3x5.8, symbol Device:C_Polarized_US
- added C49: 100nF/50V, Capacitor_SMD:C_0402_1005Metric, symbol Device:C
- added R10, R21, R22, R9: 0Ω, Resistor_SMD:R_0402_1005Metric, symbol Device:R_Small_US
- added R7: 10kΩ, Resistor_SMD:R_0402_1005Metric, symbol Device:R_US
- added S1: SSSS811101, SAVITAR:SSSS811101, symbol SAVITAR:SSSS811101
- added U2: FSUSB42MUX, SAVITAR:SOP50P490X110-10N, symbol SAVITAR:FSUSB42MUX
- C1, C2, C5, C6, C7: footprint Capacitor_SMD:C_0603_1608Metric -> Capacitor_SMD:C_0402_1005Metric
- C12: renamed from C33; footprint Capacitor_SMD:C_0603_1608Metric -> Capacitor_SMD:C_0402_1005Metric
- C13: renamed from C34; footprint Capacitor_SMD:C_0603_1608Metric -> Capacitor_SMD:C_0402_1005Metric
- C16: renamed from C36; footprint Capacitor_SMD:C_0603_1608Metric -> Capacitor_SMD:C_0402_1005Metric
- C17: renamed from C21; footprint Capacitor_SMD:C_0603_1608Metric -> Capacitor_SMD:C_0402_1005Metric
- C18: renamed from C23; footprint Capacitor_SMD:C_0603_1608Metric -> Capacitor_SMD:C_0402_1005Metric
- C19: renamed from C24; footprint Capacitor_SMD:C_0603_1608Metric -> Capacitor_SMD:C_0402_1005Metric
- C22: renamed from C42; footprint Capacitor_SMD:C_0603_1608Metric -> Capacitor_SMD:C_0402_1005Metric
- C23: renamed from C43; footprint Capacitor_SMD:C_0603_1608Metric -> Capacitor_SMD:C_0402_1005Metric
- C24: renamed from C45; footprint Capacitor_SMD:C_0603_1608Metric -> Capacitor_SMD:C_0402_1005Metric
- C25: renamed from C44; footprint Capacitor_SMD:C_0603_1608Metric -> Capacitor_SMD:C_0402_1005Metric
- C27: renamed from C47; value 22uF/25V -> 22uF/16V
- C3, C4: value 2.2uF/25V -> 2.2uF/16V; footprint Capacitor_SMD:C_0603_1608Metric -> Capacitor_SMD:C_0402_1005Metric
- C30: renamed from C16; footprint Capacitor_SMD:C_0603_1608Metric -> Capacitor_SMD:C_0402_1005Metric
- C32: renamed from C18; footprint Capacitor_SMD:C_0603_1608Metric -> Capacitor_SMD:C_0402_1005Metric
- C34: renamed from C17; value 22uF/25V -> 22uF/16V
- C35: renamed from C49; value 22uF/25V -> 22uF/16V; footprint Capacitor_SMD:C_1206_3216Metric -> Capacitor_SMD:C_0805_2012Metric
- C36: renamed from C20; footprint Capacitor_SMD:C_0603_1608Metric -> Capacitor_SMD:C_0402_1005Metric
- C37: renamed from C19; footprint Capacitor_SMD:C_0603_1608Metric -> Capacitor_SMD:C_0402_1005Metric
- C38: renamed from C22; value 22uF/25V -> 22uF/16V; footprint Capacitor_SMD:C_1206_3216Metric -> Capacitor_SMD:C_0805_2012Metric
- C39: renamed from C26; value 10uF/25V -> 10uF/16V
- C40: renamed from C30; value 2.2uF/25V -> 2.2uF/16V; footprint Capacitor_SMD:C_0603_1608Metric -> Capacitor_SMD:C_0402_1005Metric
- R1, R2: footprint Resistor_SMD:R_0603_1608Metric -> Resistor_SMD:R_0402_1005Metric
- R11: renamed from R30; footprint Resistor_SMD:R_0603_1608Metric -> Resistor_SMD:R_0402_1005Metric
- R12: renamed from R6; footprint Resistor_SMD:R_0603_1608Metric -> Resistor_SMD:R_0402_1005Metric
- R13: renamed from R8; footprint Resistor_SMD:R_0603_1608Metric -> Resistor_SMD:R_0402_1005Metric
- R14: renamed from R18; footprint Resistor_SMD:R_0603_1608Metric -> Resistor_SMD:R_0402_1005Metric
- R15: renamed from R19; footprint Resistor_SMD:R_0603_1608Metric -> Resistor_SMD:R_0402_1005Metric
- R16: renamed from R10; footprint Resistor_SMD:R_0603_1608Metric -> Resistor_SMD:R_0402_1005Metric
- R17: renamed from R4; footprint Resistor_SMD:R_0603_1608Metric -> Resistor_SMD:R_0402_1005Metric
- R18: renamed from R5; footprint Resistor_SMD:R_0603_1608Metric -> Resistor_SMD:R_0402_1005Metric
- R19: renamed from R37; footprint Resistor_SMD:R_0603_1608Metric -> Resistor_SMD:R_0402_1005Metric
- R20: renamed from R7; footprint Resistor_SMD:R_0603_1608Metric -> Resistor_SMD:R_0402_1005Metric
- R23: renamed from R11; footprint Resistor_SMD:R_0603_1608Metric -> Resistor_SMD:R_0402_1005Metric
- R24: renamed from R12; footprint Resistor_SMD:R_0603_1608Metric -> Resistor_SMD:R_0402_1005Metric
- R25: renamed from R13; footprint Resistor_SMD:R_0603_1608Metric -> Resistor_SMD:R_0402_1005Metric
- R26: renamed from R14; footprint Resistor_SMD:R_0603_1608Metric -> Resistor_SMD:R_0402_1005Metric
- R27: renamed from R15; footprint Resistor_SMD:R_0603_1608Metric -> Resistor_SMD:R_0402_1005Metric
- R28: renamed from R16; footprint Resistor_SMD:R_0603_1608Metric -> Resistor_SMD:R_0402_1005Metric
- R29: renamed from R17; footprint Resistor_SMD:R_0603_1608Metric -> Resistor_SMD:R_0402_1005Metric
- R3: renamed from R39; footprint Resistor_SMD:R_0603_1608Metric -> Resistor_SMD:R_0402_1005Metric
- R4: renamed from R40; footprint Resistor_SMD:R_0603_1608Metric -> Resistor_SMD:R_0402_1005Metric
- R5: renamed from R3; footprint Resistor_SMD:R_0603_1608Metric -> Resistor_SMD:R_0402_1005Metric
- R6: renamed from R31; footprint Resistor_SMD:R_0603_1608Metric -> Resistor_SMD:R_0402_1005Metric
- R8: renamed from R34; footprint Resistor_SMD:R_0603_1608Metric -> Resistor_SMD:R_0402_1005Metric
- SHUNT1, SHUNT2: footprint Resistor_SMD:R_1206_3216Metric -> Resistor_SMD:R_0805_2012Metric
- USBC1: renamed from J3; footprint (none) -> Connector_USB:USB_C_Receptacle_HRO_TYPE-C-31-M-12
- Y1: footprint (none) -> Crystal:Crystal_SMD_3215-2Pin_3.2x1.5mm
- renumbered C41 to C14, C35 to C15, C12 to C20, C48 to C33, SW3 to SW1, SW1 to SW2, SW2 to SW3, TPA3 to TPA1, TPA4 to TPA2, TPA5 to TPA3, TPA6 to TPA4, TPA7 to TPA5, TPA1 to TPA6, TPA2 to TPA7, U21 to U1, U20 to U3, U2 to U4, U3 to U5, U1 to UNOT1
Connections:
- net D+: now also U2.3 (D+); no longer U3.46 (PA25)
- net D-: now also U2.4 (D-); no longer U3.45 (PA24)
- net GND: now also C47.2, C48.2, C49.1, R7.2, S1.3, S1.4, S1.5, S1.6, S1.7, U2.5 (GND)
- net VBAT: now also C47.1, C48.1
- net VCC: now also S1.1, U2.1 (VCC)
- net ESP_BOOT: now reaches R24.2, SW3.2, U4.23 (IO9)
- net at U4.26 (IO18): now also R21.2
- net at U4.27 (IO19): now also R22.2
- net at FB1.2, TPA5.1, U3.8 (VDDANA): now also C49.2
- new net: R10.2, U3.46 (PA25)
- new net: R9.2, U3.45 (PA24)
- new net: R7.1, U2.10 (/OE)
- new net ESP_D+: R22.1, U2.7 (HSD1+)
- new net ESP_D-: R21.1, U2.6 (HSD1-)
- new net SAMD_D+: R10.1, U2.9 (HSD2+)
- new net SAMD_D-: R9.1, U2.8 (HSD2-)
- new net USB_SEL: S1.2 (COM), U2.2 (SEL)
- no-connect marks 35 -> 78
Other:
- note added: "1.5A × 0.050Ω = 75mV 75mV × 20 = 1.5V"
- note added: "HIGH -> SAMD51 LOW -> ESP32"
- note added: "PROGRAMMING ONLY"
- note removed: "2.5A × 0.033Ω = 82.5mV 82.5mV × 20 = 1.65V"
- note removed: "TODO: Cut between V_{USB} and V_{IN} Pad on the TEENSY 4 board."
- moved on the sheet: C12, C13, C14, C15, C16, C18, C22, C23, C24, C25, C27, C6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
