File: MCU.kicad_sch (KiCad schematic)
At the start: 96 parts, among them IC1 MT2492, J1 FH34SRJ-8S-0.5SH_50_, SW1 TS-1088-AR02016, SW2 TS-1088-AR02016, SW3 TS-1088-AR02016, U1 USBLC6-2SC6, U2 FSUSB42MUX, U3 ATSAMD51J19A-A, U4 ESP32-C3-MINI-1-H4X, U5 TLV75733PDBV, Y1 32.768kHz

Commit message: Removed the following: ESP32-C3 USB path: FSUSB4 mux + slide switch — dropped entirely. Rationale: SAMD51 programming now exclusively via SWD (Segger, no USB needed), telemetry/config now exclusively via ESP32 dashboard. Nothing on SAMD51 side needed USB anymore, so the mux had nothing left to arbitrate. USB-C D+/D− now routes straight to ESP32-C3 GPIO18/19 (native USB-Serial/JTAG) through USBLC6 only. SAMD51 reset debounce network (C15, R8) — removed. R11 (10k pull-up) + SW1 remain, button now wired directly RESET-to-GND with no RC filtering. Accepted tradeoff: possible 2–3x reset pulses on switch bounce, functionally harmless on SAMD51. Kept components: SAMD51 reset button itself stays populated — this is the field/competition-floor recovery path when not tethered to Segger, distinct from Segger's own nRESET (session-only, tethered). Consistent with uptime priority. SWD 5-pin header (VTref/GND/SWCLK/SWDIO/RESET) confirmed sufficient for full SAMD51 programming/debug on battery power alone — no USB dependency, no bootloader entry sequence. ESP32-C3 auto-reset via native USB-Serial/JTAG confirmed real (esptool usb-reset path) — no transistor/DTR-RTS network needed. EN (10k+cap) and GPIO9 (10k pull-up) support components still required regardless; only the manual buttons and transistor auto-reset circuit are removable.
Parts:
- removed C12, C13: 18pF/25V, Capacitor_SMD:C_0402_1005Metric, symbol Device:C
- removed C15: 1uF/16V, Capacitor_SMD:C_0603_1608Metric, symbol Device:C
- removed R10, R9: 0Ω, Resistor_SMD:R_0402_1005Metric, symbol Device:R_Small_US
- removed R7: 10kΩ, Resistor_SMD:R_0402_1005Metric, symbol Device:R_US
- removed R8: 330Ω, Resistor_SMD:R_0402_1005Metric, symbol Device:R_Small_US
- removed S1: SSSS811101, SAVITAR:SSSS811101, symbol SAVITAR:SSSS811101
- removed SW2, SW3: TS-1088-AR02016, Button_Switch_SMD:SW_SPST_TS-1088-xR020, symbol Switch:SW_Push
- removed TPA1, TPA2, TPA3, TPA4, TPA5: TestPoint, TestPoint:TestPoint_THTPad_D2.0mm_Drill1.0mm, symbol Connector:TestPoint
- removed U2: FSUSB42MUX, SAVITAR:SOP50P490X110-10N, symbol SAVITAR:FSUSB42MUX
- removed Y1: 32.768kHz, Crystal:Crystal_SMD_3215-2Pin_3.2x1.5mm, symbol Device:Crystal
- added ESP_JMP1, ESP_JMP2: TestPoint, symbol Connector:TestPoint
- added R44: 10kΩ, Resistor_SMD:R_0402_1005Metric, symbol Device:R_US
- added SWD_CLK, SWD_GND, SWD_IO, SWD_PWR, SWD_RST: TestPoint, TestPoint:TestPoint_THTPad_D2.0mm_Drill1.0mm, symbol Connector:TestPoint
Connections:
- net D+ is gone; now on net ESP_D+: U1.4 (I/O2)
- net D- is gone; now on net ESP_D-: U1.6 (I/O1)
- net ESP_BOOT: now also ESP_JMP1.1
- net GND: now also C49.2, ESP_JMP2.1, SWD_GND.1; no longer C49.1
- net SWCLK: now also SWD_CLK.1
- net SWDIO: now also SWD_IO.1
- net VCC: now also R44.1
- net SWD5: now reaches SW1.2
- net SWD5: now also R11.2, U3.52 (~{RESET}), SWD_RST.1
- net at U4.5 (IO2): now also R44.2
- net SWD1: now reaches FB1.2, U3.8 (VDDANA)
- net SWD1: now also C49.1, SWD_PWR.1; no longer C49.2
- no-connect marks 78 -> 81
Other:
- note added: "Checklist - No need for RTC so no OSC on either MCU - SAMD51 - Automatic reset is done over Native USB"
- note added: "ESP32-C3"
- note added: "STRAPPING PINS: GPIO2 GPIO8 GPIO9"
- note removed: "ESP32-C3-MINI-1"
- note removed: "HIGH -> SAMD51 LOW -> ESP32"
- moved on the sheet: C32, C35, C38, C49, FB1, R11, R3, R4, R6, SW1, U1, USBC1
