File: MCU.kicad_sch (KiCad schematic)
At the start: 79 parts, among them IC1 MT2492, J1 FH34SRJ-8S-0.5SH_50_, SW1 TS-1088-AR02016, U1 USBLC6-2SC6, U3 ATSAMD51J19A-A, U4 ESP32-C3-MINI-1-H4X, U5 TLV75733PDBV

Commit message: Will add info in a later commit
Parts:
- removed J1: FH34SRJ-8S-0.5SH_50_, SAVITAR:FH34SRJ8S05SH50, symbol SAVITAR:FH34SRJ-8S-0.5SH_50_
- added FPC2: FPC-05F-22PH20, EasyEDA:FPC-SMD_22P-P0.50_FPC-05F-22PH20, symbol EasyEDA:FPC-05F-22PH20
- added TP1, TP2: TestPoint, TestPoint:TestPoint_THTPad_D2.0mm_Drill1.0mm, symbol Connector:TestPoint
- FB1: value 50mΩ 2A -> 380mΩ 500mA
- renumbered C14 to C1, C24 to C10, C25 to C11, C27 to C12, C17 to C13, C18 to C14, C19 to C15, C20 to C16, C47 to C17, C32 to C18, C30 to C19, C5 to C2, C35 to C20, C36 to C21, C33 to C22, C38 to C23, C34 to C24, C37 to C25, C39 to C26, C40 to C27, C6 to C3, C7 to C4, C16 to C5, C48 to C6, C49 to C7, C22 to C8, C23 to C9, R14 to R10, R15 to R11, R16 to R12, R17 to R13, R18 to R14, R21 to R15, R22 to R16, R23 to R17, R19 to R18, R20 to R19, R24 to R20, R25 to R21, R26 to R22, R44 to R23, R27 to R24, R28 to R25, R29 to R26, R5 to R3, R6 to R4, R11 to R5, R3 to R6, R4 to R7, R12 to R8, R13 to R9, SWD_CLK to SWD_CLK1, SWD_GND to SWD_GND1, SWD_IO to SWD_IO1, SWD_PWR to SWD_PWR1, SWD_RST to SWD_RST1, TPA6 to TPA1, TPA7 to TPA2, U3 to U2, U4 to U3, U5 to U4
Connections:
- net GND: now also FPC2.1, FPC2.23, FPC2.24, TP2.1
- net VBAT: now also TP1.1
- net VCC: now also FPC2.2
- net SWD1 renamed VCCANA
- new net A0: FPC2.19
- new net A1: FPC2.20
- new net A2: FPC2.21
- new net EN: FPC2.22
- new net S0: FPC2.3
- new net S1: FPC2.4
- new net S10: FPC2.13
- new net S11: FPC2.14
- new net S12: FPC2.15
- new net S13: FPC2.16
- new net S14: FPC2.17
- new net S15: FPC2.18
- new net S2: FPC2.5
- new net S3: FPC2.6
- new net S4: FPC2.7
- new net S5: FPC2.8
- new net S6: FPC2.9
- new net S7: FPC2.10
- new net S8: FPC2.11
- new net S9: FPC2.12
Other:
- moved on the sheet: C18, C20, C21, C23, ESP_JMP1, ESP_JMP2, R15, R16, R17, R20, R21, R22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

Commit message: Assigned Pins on SAMD51 using Pin Planner and PMODE is hardwired to VCC (PWM mode).
Parts:
- removed UNOT1: TEENSY 4.0, SAVITAR:MODULE_DEV-15583, symbol SAVITAR:DEV-15583
Connections:
- net A0 is gone; now on net SEN_A0: FPC2.19
- net A1 is gone; now on net SEN_A1: FPC2.20
- net A2 is gone; now on net SEN_A2: FPC2.21
- net EN is gone; now on net SEN_EN: FPC2.22
- net S0 is gone; now on net SEN_S0: FPC2.3
- net S1 is gone; now on net SEN_S1: FPC2.4
- net S10 is gone; now on net SEN_S10: FPC2.13
- net S11 is gone; now on net SEN_S11: FPC2.14
- net S12 is gone; now on net SEN_S12: FPC2.15
- net S13 is gone; now on net SEN_S13: FPC2.16
- net S14 is gone; now on net SEN_S14: FPC2.17
- net S15 is gone; now on net SEN_S15: FPC2.18
- net S2 is gone; now on net SEN_S2: FPC2.5
- net S3 is gone; now on net SEN_S3: FPC2.6
- net S4 is gone; now on net SEN_S4: FPC2.7
- net S5 is gone; now on net SEN_S5: FPC2.8
- net S6 is gone; now on net SEN_S6: FPC2.9
- net S7 is gone; now on net SEN_S7: FPC2.10
- net S8 is gone; now on net SEN_S8: FPC2.11
- net S9 is gone; now on net SEN_S9: FPC2.12
- net SAMD_RX1 is gone; now on net ESP_TX: R22.1
- net SAMD_TX1 is gone; now on net ESP_RX: R21.1
- net SENSE_IN_A1 is gone; now on net MOT_A1: DRV1.8 (OUT1)
- net SENSE_IN_B1 is gone; now on net MOT_B1: DRV2.8 (OUT1)
- net BAT_LEVEL: now also U2.63 (PB02)
- net MOT_A.C_STALL: now also U2.61 (PB00)
- net MOT_A.EN/IN1: now also U2.37 (PA18)
- net MOT_A.PH/IN2: now also U2.38 (PA19)
- net MOT_A.~{FAULT}: now also U2.36 (PA17)
- net MOT_A.~{SLEEP}: now also U2.35 (PA16)
- net MOT_B.C_STALL: now also U2.62 (PB01)
- net MOT_B.EN/IN1: now also U2.43 (PA22)
- net MOT_B.PH/IN2: now also U2.44 (PA23)
- net MOT_B.~{FAULT}: now also U2.60 (PB31)
- net MOT_B.~{SLEEP}: now also U2.59 (PB30)
- net SEN_EN: now also U2.2 (PA01)
- net SEN_S0: now also U2.3 (PA02)
- net SEN_S1: now also U2.4 (PA03)
- net SEN_S2: now also U2.13 (PA04)
- net STATUS_LED: now also U2.28 (PB15)
- net SEN_S8: now reaches U2.10 (PB07)
- net SEN_S15: now reaches U2.11 (PB08)
- net SEN_S14: now reaches U2.12 (PB09)
- net SEN_S3: now reaches U2.14 (PA05)
- net SEN_S4: now reaches U2.15 (PA06)
- net SEN_S5: now reaches U2.16 (PA07)
- net SEN_S13: now reaches U2.17 (PA08)
- net SEN_S12: now reaches U2.18 (PA09)
- net SEN_S6: now reaches U2.19 (PA10)
- net SEN_S7: now reaches U2.20 (PA11)
- net SEN_A0: now reaches U2.25 (PB12)
- net SEN_A1: now reaches U2.26 (PB13)
- net SEN_A2: now reaches U2.27 (PB14)
- net ESP_TX: now reaches U2.29 (PA12)
- net ESP_RX: now reaches U2.30 (PA13)
- net SEN_S11: now reaches U2.5 (PB04)
- net SEN_S10: now reaches U2.6 (PB05)
- net SEN_S9: now reaches U2.9 (PB06)
- net MOT_A.PMODE: no longer names the net of DRV1.16 (PMODE), R3.2
- net MOT_B.PMODE: no longer names the net of DRV2.16 (PMODE), R12.2
- no-connect marks 79 -> 40
Other:
- note added: "ADC0"
- note added: "ADC1"
- note added: "FOOTPRINT CONNECTOR"
- note added: "MOT_A"
- note added: "MOT_B"
- note added: "TCC1"
- note removed: "TEENSY 4"
- note removed: "V_{IN} = 3.6V .. 5.5V"
- moved on the sheet: R4

Commit message: Updated
Parts:
- FPC2: footprint EasyEDA:FPC-SMD_22P-P0.50_FPC-05F-22PH20 -> easyeda2kicad:FPC-SMD_22P-P0.50_FPC-05F-22PH20
Connections:
- net ANODE1: now reaches D1.2 (A), R10.2
- net IO8: now reaches R24.2, U3.22 (IO8)
- net USB_D-: now reaches U1.1 (I/O1), USBC1.A7 (D-), USBC1.B7 (D-)
- net USB_D+: now reaches U1.3 (I/O2), USBC1.A6 (D+), USBC1.B6 (D+)
- net IO18: now reaches R15.2, U3.26 (IO18)
- net IO19: now reaches R16.2, U3.27 (IO19)
- net RX: now reaches R25.2, U3.30 (RXD0)
- net TX: now reaches R26.2, U3.31 (TXD0)
- net IO2: now reaches R23.2, U3.5 (IO2)
- net CC2: now reaches R7.2, USBC1.B5 (CC2)
- net PMODE_B: now reaches DRV2.16 (PMODE), R12.2
- net PMODE_A: now reaches DRV1.16 (PMODE), R3.2
- net CC1: now reaches R6.2, USBC1.A5 (CC1)
- net FB: now reaches C22.1, IC1.3 (FB), R18.2, R19.1
- net VCP_A: now reaches C2.2, DRV1.12 (VCP)
- net CPL_A: now reaches C4.1, DRV1.13 (CPH)
- net CPL_A: now also C4.2, DRV1.14 (CPL)
- net CPH_B: now reaches C15.1, DRV2.13 (CPH)
- net CPL_B: now reaches C15.2, DRV2.14 (CPL)
- net VCP_B: now reaches C13.2, DRV2.12 (VCP)
- net ANODE2: now reaches D2.2 (A), R11.2
- net SWD5 renamed RST
Other:
- note added: "SENSOR"
- note removed: "FOOTPRINT CONNECTOR"
- moved on the sheet: C21, D1, D2, R12, R2, R3
