File: SAVITAR_V2.kicad_pcb (KiCad board)
At the start: 2 copper layers, 127.1 x 19.1 mm, 71 parts, among them IC1 CD4051BM_TR, IC2 CD4051BM_TR, J2 FH34SRJ-12S-0.5SH_50_

Commit message: Added dedicated Current Sensing IC INA240. Changed Buck output from 3.8V (edge of Teensy's LDO supply voltage) to 5V.
Parts:
- removed IC1, IC2: CD4051BM_TR, CD4051BM_TR:SOIC127P602X182-16N
- removed J2: FH34SRJ-12S-0.5SH_50_, FH34SRJ-12S-0.5SH_50_:FH34SRJ12S05SH50
- removed LED1, LED2, LEDQ1, LEDQ10, LEDQ11, LEDQ12, LEDQ13, LEDQ14, LEDQ15, LEDQ16, LEDQ2, LEDQ3, LEDQ4, LEDQ5, LEDQ6, LEDQ7, LEDQ8, LEDQ9: XL-1608SURC-06, LED_SMD:LED_0603_1608Metric
- removed R1, R17, R18, R19, R2, R20, R21, R22, R23, R24, R3, R4, R5, R6, R7, R8: 100Ω, Resistor_SMD:R_0603_1608Metric
- removed R10, R11, R12, R13, R14, R15, R16, R25, R26, R27, R28, R29, R30, R31, R32, R9: 47kΩ, Resistor_SMD:R_0603_1608Metric
- removed RL1, RL2: 1kΩ, Resistor_SMD:R_0603_1608Metric
- removed S1, S10, S11, S12, S13, S14, S15, S16, S2, S3, S4, S5, S6, S7, S8, S9: QRE1113GR, OptoDevice:OnSemi_CASE100CY
Other:
- board outline removed

Commit message: Added 3D models to third party footprints. Final Teensy version, switching to SAMD51 custom setup. Please add tag.
Parts:
- added C1: 100nF/50V, Capacitor_SMD:C_0603_1608Metric, F.Cu at (44.2, 116.6)
- added C10: 100nF/50V, Capacitor_SMD:C_0603_1608Metric, F.Cu at (44.2, 134.1)
- added C11: 47uF, Capacitor_SMD:C_1206_3216Metric, F.Cu at (39.4, 123.7)
- added C12: 22uF/25V, Capacitor_SMD:C_0805_2012Metric, F.Cu at (64.4, 156.6)
- added C13: 2.2uF/25V, Capacitor_SMD:C_0603_1608Metric, F.Cu at (48.2, 116.6)
- added C14: 47uF/25V, Capacitor_SMD:C_1206_3216Metric, F.Cu at (39.4, 127.0)
- added C15: 47uF/25V, Capacitor_SMD:C_1206_3216Metric, F.Cu at (39.4, 130.4)
- added C16: 22nF/50V, Capacitor_SMD:C_0603_1608Metric, F.Cu at (48.2, 119.1)
- added C17: 22uF/25V, LED_SMD:LED_0805_2012Metric, F.Cu at (44.4, 163.5)
- added C18: 100nF/50V, Capacitor_SMD:C_0603_1608Metric, F.Cu at (48.2, 121.6)
- added C19: 100nF/50V, Capacitor_SMD:C_0603_1608Metric, F.Cu at (48.2, 124.1)
- added C2: 100nF/50V, Capacitor_SMD:C_0603_1608Metric, F.Cu at (44.2, 119.1)
- added C20: 1uF/16V, Capacitor_SMD:C_0603_1608Metric, F.Cu at (48.2, 126.6)
- added C21: 100nF/16V, Capacitor_SMD:C_0603_1608Metric, F.Cu at (48.2, 129.1)
- added C22: 22uF/25V, Capacitor_SMD:C_1206_3216Metric, F.Cu at (39.4, 133.7)
- added C23: 100nF/50V, Capacitor_SMD:C_0603_1608Metric, F.Cu at (48.2, 131.6)
- added C24: 22nF/50V, Capacitor_SMD:C_0603_1608Metric, F.Cu at (48.2, 134.1)
- added C25: 47uF, Capacitor_SMD:C_1206_3216Metric, F.Cu at (39.4, 137.1)
- added C26: 10uF/25V, Capacitor_SMD:C_0603_1608Metric, F.Cu at (52.2, 116.6)
- added C27: 47uF, Capacitor_SMD:C_1206_3216Metric, F.Cu at (39.4, 140.4)
- added C28: 47uF, Capacitor_SMD:C_1206_3216Metric, F.Cu at (39.4, 143.8)
- added C29: 47uF/25V, Capacitor_SMD:C_1206_3216Metric, F.Cu at (39.4, 147.1)
- added C3: 2.2uF/25V, Capacitor_SMD:C_0603_1608Metric, F.Cu at (44.2, 121.6)
- added C30: 2.2uF/25V, Capacitor_SMD:C_0603_1608Metric, F.Cu at (52.2, 119.1)
- added C31: 100nF/50V, Capacitor_SMD:C_0603_1608Metric, F.Cu at (44.8, 33.9)
- added C32: 1uF/25V, Capacitor_SMD:C_0603_1608Metric, F.Cu at (44.8, 36.4)
- added C37: 100nF, Capacitor_SMD:C_0603_1608Metric, F.Cu at (44.8, 38.9)
- added C38: 100nF, Capacitor_SMD:C_0603_1608Metric, F.Cu at (44.8, 41.4)
- added C39: 100nF, Capacitor_SMD:C_0603_1608Metric, F.Cu at (44.8, 44.0)
- added C4: 2.2uF/25V, Capacitor_SMD:C_0603_1608Metric, F.Cu at (44.2, 124.1)
- added C40: 100nF/50V, Capacitor_SMD:C_0603_1608Metric, F.Cu at (48.8, 33.9)
- added C5: 100nF/16V, Capacitor_SMD:C_0603_1608Metric, F.Cu at (44.2, 126.6)
- added C6: 100nF/50V, Capacitor_SMD:C_0603_1608Metric, F.Cu at (44.2, 129.1)
- added C7: 22nF/50V, Capacitor_SMD:C_0603_1608Metric, F.Cu at (44.2, 131.6)
- added C8: 47uF, Capacitor_SMD:C_1206_3216Metric, F.Cu at (39.4, 117.0)
- added C9: 47uF, Capacitor_SMD:C_1206_3216Metric, F.Cu at (39.4, 120.3)
- added D1: SML-D12D8WT86, LED_SMD:LED_0603_1608Metric, F.Cu at (59.0, 160.9)
- added D2: SML-D12D8WT86, LED_SMD:LED_0603_1608Metric, F.Cu at (59.0, 163.5)
- added D3: SML-D12D8WT86, LED_SMD:LED_0603_1608Metric, F.Cu at (56.7, 14.7)
- added D4: SML-D12D8WT86, LED_SMD:LED_0603_1608Metric, F.Cu at (56.7, 17.2)
- added DEMUX1: 74HC238D,653, SAVITAR:74HC238D653, F.Cu at (32.4, 49.5)
- added DRV1: DRV8874PWPR, SAVITAR:SOP65P640X155-18N, F.Cu at (62.9, 139.6)
- added DRV2: DRV8874PWPR, SAVITAR:SOP65P640X155-18N, F.Cu at (62.9, 147.9)
- added IC1: MT2492, SAVITAR:SOT95P280X145-6N, F.Cu at (59.5, 157.4)
- added INAA1: INA240A1DR, SAVITAR:SOIC127P600X175-8N, F.Cu at (21.5, 156.4)
- added INAB1: INA240A1DR, SAVITAR:SOIC127P600X175-8N, F.Cu at (21.5, 162.9)
- added J1: FH34SRJ-8S-0.5SH_50_, SAVITAR:FH34SRJ8S05SH50, F.Cu at (38.5, 156.5)
- added J2: FH34SRJ-8S-0.5SH_50_, SAVITAR:FH34SRJ8S05SH50, F.Cu at (47.3, 48.7)
- added L1: 22uH, Inductor_SMD:L_1210_3225Metric, F.Cu at (54.1, 163.8)
- added MUX1: 74HC4051, Package_SO:SOIC-16_3.9x9.9mm_P1.27mm, F.Cu at (30.1, 38.6)
- added MUX2: 74HC4051, Package_SO:SOIC-16_3.9x9.9mm_P1.27mm, F.Cu at (38.5, 38.6)
- added NMOS1: TBD62083AFNG_Z,EL_, SAVITAR:SOP65P640X155-18N, F.Cu at (62.5, 51.8)
- added Q1: MMBT3904, Package_TO_SOT_SMD:SOT-23, F.Cu at (57.1, 20.8)
- added R1: 2.87kΩ(1%), Resistor_SMD:R_0603_1608Metric, F.Cu at (52.2, 121.6)
- added R10: 10kΩ, Resistor_SMD:R_0603_1608Metric, F.Cu at (56.2, 124.1)
- added R11: 10kΩ(1%), Resistor_SMD:R_0603_1608Metric, F.Cu at (56.2, 126.6)
- added R12: 10kΩ, Resistor_SMD:R_0603_1608Metric, F.Cu at (56.2, 129.1)
- added R13: 470Ω, Resistor_SMD:R_0603_1608Metric, F.Cu at (56.2, 131.6)
- added R14: 470Ω, Resistor_SMD:R_0603_1608Metric, F.Cu at (56.2, 134.1)
- added R15: 10kΩ, Resistor_SMD:R_0603_1608Metric, F.Cu at (60.2, 116.6)
- added R16: 0Ω, Resistor_SMD:R_0603_1608Metric, F.Cu at (60.2, 119.1)
- added R17: 0Ω, Resistor_SMD:R_0603_1608Metric, F.Cu at (60.2, 121.6)
- added R18: 510Ω, Resistor_SMD:R_0603_1608Metric, F.Cu at (60.2, 124.1)
- added R19: 510Ω, Resistor_SMD:R_0603_1608Metric, F.Cu at (60.2, 126.6)
- added R2: 10kΩ, Resistor_SMD:R_0603_1608Metric, F.Cu at (52.2, 124.1)
- added R20: 33Ω, Resistor_SMD:R_0603_1608Metric, F.Cu at (48.8, 36.4)
- added R21: 33Ω, Resistor_SMD:R_0603_1608Metric, F.Cu at (48.8, 38.9)
- added R22: 33Ω, Resistor_SMD:R_0603_1608Metric, F.Cu at (48.8, 41.4)
- added R23: 33Ω, Resistor_SMD:R_0603_1608Metric, F.Cu at (48.8, 44.0)
- added R24: 510Ω, Resistor_SMD:R_0603_1608Metric, F.Cu at (52.8, 33.9)
- added R25: 510Ω, Resistor_SMD:R_0603_1608Metric, F.Cu at (52.8, 36.4)
- added R26: 33Ω, Resistor_SMD:R_0603_1608Metric, F.Cu at (52.8, 38.9)
- added R27: 33Ω, Resistor_SMD:R_0603_1608Metric, F.Cu at (52.8, 41.4)
- added R28: 33Ω, Resistor_SMD:R_0603_1608Metric, F.Cu at (52.8, 44.0)
- added R29: 33Ω, Resistor_SMD:R_0603_1608Metric, F.Cu at (56.8, 33.9)
- added R3: 10kΩ, Resistor_SMD:R_0603_1608Metric, F.Cu at (52.2, 126.6)
- added R32: 10kΩ, Resistor_SMD:R_0603_1608Metric, F.Cu at (56.8, 36.4)
- added R33: 10kΩ, Resistor_SMD:R_0603_1608Metric, F.Cu at (56.8, 38.9)
- added R35: 47kΩ, Resistor_SMD:R_0603_1608Metric, F.Cu at (56.8, 41.4)
- added R36: 47kΩ, Resistor_SMD:R_0603_1608Metric, F.Cu at (56.8, 44.0)
- added R4: 100kΩ(1%), Resistor_SMD:R_0603_1608Metric, F.Cu at (52.2, 129.1)
- added R5: 33kΩ(1%), Resistor_SMD:R_0603_1608Metric, F.Cu at (52.2, 131.6)
- added R6: 2.87kΩ(1%), Resistor_SMD:R_0603_1608Metric, F.Cu at (52.2, 134.1)
- added R7: 13.7kΩ(1%), Resistor_SMD:R_0603_1608Metric, F.Cu at (56.2, 116.6)
- added R8: 10kΩ, Resistor_SMD:R_0603_1608Metric, F.Cu at (56.2, 119.1)
- added R9: 100kΩ(1%), Resistor_SMD:R_0603_1608Metric, F.Cu at (56.2, 121.6)
- added SHUNT1: 33mΩ, Resistor_SMD:R_1206_3216Metric, F.Cu at (54.1, 156.8)
- added SHUNT2: 33mΩ, Resistor_SMD:R_1206_3216Metric, F.Cu at (54.1, 160.1)
- added SWB1: TS-1088-AR02016, Button_Switch_SMD:SW_SPST_TS-1088-xR020, F.Cu at (29.2, 155.4)
- added SWEN1: TS-1088-AR02016, Button_Switch_SMD:SW_SPST_TS-1088-xR020, F.Cu at (29.2, 159.9)
- added TPA1: TestPoint, TestPoint:TestPoint_THTPad_2.0x2.0mm_Drill1.0mm, F.Cu at (64.3, 117.3)
- added TPA2: TestPoint, TestPoint:TestPoint_THTPad_2.0x2.0mm_Drill1.0mm, F.Cu at (64.3, 121.4)
- added TPB1: TestPoint, TestPoint:TestPoint_THTPad_2.0x2.0mm_Drill1.0mm, F.Cu at (64.3, 125.4)
- added TPB2: TestPoint, TestPoint:TestPoint_THTPad_2.0x2.0mm_Drill1.0mm, F.Cu at (64.3, 129.5)
- added U1: TEENSY 4.0, SAVITAR:MODULE_DEV-15583, F.Cu at (111.3, 120.4)
- added U10: QRE1113GR, OptoDevice:OnSemi_CASE100CY, F.Cu at (36.7, 25.4)
- added U11: QRE1113GR, OptoDevice:OnSemi_CASE100CY, F.Cu at (36.7, 30.2)
- added U12: QRE1113GR, OptoDevice:OnSemi_CASE100CY, F.Cu at (43.9, 15.7)
- added U13: QRE1113GR, OptoDevice:OnSemi_CASE100CY, F.Cu at (43.9, 20.6)
- added U14: QRE1113GR, OptoDevice:OnSemi_CASE100CY, F.Cu at (43.9, 25.4)
- added U15: QRE1113GR, OptoDevice:OnSemi_CASE100CY, F.Cu at (43.9, 30.2)
- added U16: QRE1113GR, OptoDevice:OnSemi_CASE100CY, F.Cu at (51.1, 15.7)
- added U17: QRE1113GR, OptoDevice:OnSemi_CASE100CY, F.Cu at (51.1, 20.6)
- added U18: QRE1113GR, OptoDevice:OnSemi_CASE100CY, F.Cu at (51.1, 25.4)
- added U19: QRE1113GR, OptoDevice:OnSemi_CASE100CY, F.Cu at (51.1, 30.2)
- added U2: ESP32-C3-MINI-1-H4X, SAVITAR:ESP32C3MINI1H4X, F.Cu at (50.3, 145.2)
- added U3: TLV75733PDBV, Package_TO_SOT_SMD:SOT-23-5, F.Cu at (63.5, 162.0)
- added U4: QRE1113GR, OptoDevice:OnSemi_CASE100CY, F.Cu at (89.2, 40.0)
- added U5: QRE1113GR, OptoDevice:OnSemi_CASE100CY, F.Cu at (29.5, 20.6)
- added U6: QRE1113GR, OptoDevice:OnSemi_CASE100CY, F.Cu at (29.5, 25.4)
- added U7: QRE1113GR, OptoDevice:OnSemi_CASE100CY, F.Cu at (29.5, 30.2)
- added U8: QRE1113GR, OptoDevice:OnSemi_CASE100CY, F.Cu at (99.3, 40.0)
- added U9: QRE1113GR, OptoDevice:OnSemi_CASE100CY, F.Cu at (36.7, 20.6)
Other:
- board outline added: 127.2 x 119.8 mm

Commit message: Made passives smaller from 0603 to 0402 because I will solder them with hot air gun anyway. Started positioning SAMD51 bypass caps.
Parts:
- removed C26: 10uF/25V, Capacitor_SMD:C_0603_1608Metric
- removed SWB1, SWEN1: TS-1088-AR02016, Button_Switch_SMD:SW_SPST_TS-1088-xR020
- added C33: 22pF, Capacitor_SMD:C_0603_1608Metric, F.Cu at (86.1, 137.5)
- added C34: 22uF/16V, LED_SMD:LED_0805_2012Metric, F.Cu at (59.0, 188.4)
- added C35: 22uF/16V, Capacitor_SMD:C_0805_2012Metric, F.Cu at (95.2, 184.8)
- added C36: 1uF/16V, Capacitor_SMD:C_0402_1005Metric, F.Cu at (86.1, 140.0)
- added C41: 100nF/50V, Capacitor_SMD:C_0402_1005Metric, F.Cu at (133.0, 151.8)
- added C42: 1uF/16V, Capacitor_SMD:C_0402_1005Metric, F.Cu at (133.0, 154.3)
- added C43: 100nF, Capacitor_SMD:C_0402_1005Metric, F.Cu at (133.0, 156.8)
- added C44: 100nF, Capacitor_SMD:C_0402_1005Metric, F.Cu at (133.0, 159.3)
- added C45: 100nF, Capacitor_SMD:C_0402_1005Metric, F.Cu at (133.0, 161.8)
- added C46: 100nF/50V, Capacitor_SMD:C_0402_1005Metric, F.Cu at (137.0, 151.8)
- added C47: 100uF/25V, Capacitor_SMD:CP_Elec_6.3x5.8, F.Cu at (131.1, 196.9)
- added C48: 100uF/25V, Capacitor_SMD:CP_Elec_6.3x5.8, F.Cu at (131.1, 205.0)
- added C49: 100nF/50V, Capacitor_SMD:C_0402_1005Metric, F.Cu at (198.6, 185.2)
- added FB1: 50mΩ 2A, Inductor_SMD:L_0603_1608Metric, F.Cu at (197.3, 186.6)
- added R30: 33Ω, Resistor_SMD:R_0402_1005Metric, F.Cu at (137.0, 154.3)
- added R31: 33Ω, Resistor_SMD:R_0402_1005Metric, F.Cu at (137.0, 156.8)
- added R34: 510Ω, Resistor_SMD:R_0402_1005Metric, F.Cu at (141.0, 151.8)
- added R37: 33Ω, Resistor_SMD:R_0402_1005Metric, F.Cu at (141.0, 159.3)
- added R38: 33Ω, Resistor_SMD:R_0402_1005Metric, F.Cu at (141.0, 161.8)
- added R39: 33Ω, Resistor_SMD:R_0402_1005Metric, F.Cu at (145.0, 151.8)
- added R40: 47kΩ, Resistor_SMD:R_0402_1005Metric, F.Cu at (145.0, 154.3)
- added R41: 10kΩ, Resistor_SMD:R_0402_1005Metric, F.Cu at (145.0, 156.8)
- added R42: 47kΩ, Resistor_SMD:R_0402_1005Metric, F.Cu at (145.0, 159.3)
- added R43: 10kΩ, Resistor_SMD:R_0402_1005Metric, F.Cu at (145.0, 161.8)
- added S1: SSSS811101, SAVITAR:SSSS811101, F.Cu at (69.5, 173.6)
- added SW1: TS-1088-AR02016, Button_Switch_SMD:SW_SPST_TS-1088-xR020, F.Cu at (60.2, 171.3)
- added SW2: TS-1088-AR02016, Button_Switch_SMD:SW_SPST_TS-1088-xR020, F.Cu at (60.2, 175.8)
- added SW3: TS-1088-AR02016, Button_Switch_SMD:SW_SPST_TS-1088-xR020, F.Cu at (60.2, 180.4)
- added TPA3: TestPoint, TestPoint:TestPoint_THTPad_D2.0mm_Drill1.0mm, F.Cu at (103.5, 204.3)
- added TPA4: TestPoint, TestPoint:TestPoint_THTPad_D2.0mm_Drill1.0mm, F.Cu at (107.6, 196.2)
- added TPA5: TestPoint, TestPoint:TestPoint_THTPad_D2.0mm_Drill1.0mm, F.Cu at (107.6, 200.3)
- added TPA6: TestPoint, TestPoint:TestPoint_THTPad_2.0x2.0mm_Drill1.0mm, F.Cu at (107.6, 204.3)
- added TPA7: TestPoint, TestPoint:TestPoint_THTPad_2.0x2.0mm_Drill1.0mm, F.Cu at (111.6, 196.2)
- added U20: QRE1113GR, OptoDevice:OnSemi_CASE100CY, F.Cu at (139.3, 143.2)
- added U21: QRE1113GR, OptoDevice:OnSemi_CASE100CY, F.Cu at (139.3, 148.0)
- added UNOT1: TEENSY 4.0, SAVITAR:MODULE_DEV-15583, F.Cu at (-175.0, 39.0)
- added USBC1: USB_C_Receptacle_USB2.0_16P, Connector_USB:USB_C_Receptacle_HRO_TYPE-C-31-M-12, F.Cu at (205.5, 210.6)
- added Y1: 32.768kHz, Crystal:Crystal_SMD_3215-2Pin_3.2x1.5mm, F.Cu at (196.9, 181.8)
- C1, C18, C2, C5, C6, C7: footprint Capacitor_SMD:C_0603_1608Metric -> Capacitor_SMD:C_0402_1005Metric
- C10: value 100nF/50V -> 47uF; footprint Capacitor_SMD:C_0603_1608Metric -> Capacitor_SMD:C_1206_3216Metric
- C11: value 47uF -> 47uF/25V
- C12: value 22uF/25V -> 18pF/25V; footprint Capacitor_SMD:C_0805_2012Metric -> Capacitor_SMD:C_0402_1005Metric
- C13: value 2.2uF/25V -> 18pF/25V; footprint Capacitor_SMD:C_0603_1608Metric -> Capacitor_SMD:C_0402_1005Metric
- C14: value 47uF/25V -> 10uF (X7R); footprint Capacitor_SMD:C_1206_3216Metric -> Capacitor_SMD:C_0603_1608Metric
- C15: value 47uF/25V -> 1uF/16V; footprint Capacitor_SMD:C_1206_3216Metric -> Capacitor_SMD:C_0603_1608Metric
- C16: value 22nF/50V -> 1uF (X7R); footprint Capacitor_SMD:C_0603_1608Metric -> Capacitor_SMD:C_0402_1005Metric
- C17: value 22uF/25V -> 100nF/16V; footprint LED_SMD:LED_0805_2012Metric -> Capacitor_SMD:C_0402_1005Metric
- C19: value 100nF/50V -> 22nF/50V; footprint Capacitor_SMD:C_0603_1608Metric -> Capacitor_SMD:C_0402_1005Metric
- C20: value 1uF/16V -> 22uF/25V; footprint Capacitor_SMD:C_0603_1608Metric -> Capacitor_SMD:C_0805_2012Metric
- C21: value 100nF/16V -> 47uF; footprint Capacitor_SMD:C_0603_1608Metric -> Capacitor_SMD:C_1206_3216Metric
- C22: value 22uF/25V -> 100nF (X7R); footprint Capacitor_SMD:C_1206_3216Metric -> Capacitor_SMD:C_0402_1005Metric
- C23: value 100nF/50V -> 100nF; footprint Capacitor_SMD:C_0603_1608Metric -> Capacitor_SMD:C_0402_1005Metric
- C24: value 22nF/50V -> 100nF; footprint Capacitor_SMD:C_0603_1608Metric -> Capacitor_SMD:C_0402_1005Metric
- C25: value 47uF -> 100nF; footprint Capacitor_SMD:C_1206_3216Metric -> Capacitor_SMD:C_0402_1005Metric
- C27: value 47uF -> 22uF/16V; footprint Capacitor_SMD:C_1206_3216Metric -> Capacitor_SMD:C_0805_2012Metric
- C29: value 47uF/25V -> 47uF
- C3, C4: value 2.2uF/25V -> 2.2uF/16V; footprint Capacitor_SMD:C_0603_1608Metric -> Capacitor_SMD:C_0402_1005Metric
- C30: value 2.2uF/25V -> 22nF/50V; footprint Capacitor_SMD:C_0603_1608Metric -> Capacitor_SMD:C_0402_1005Metric
- C31: value 100nF/50V -> 47uF/25V; footprint Capacitor_SMD:C_0603_1608Metric -> Capacitor_SMD:C_1206_3216Metric
- C32: value 1uF/25V -> 100nF/50V; footprint Capacitor_SMD:C_0603_1608Metric -> Capacitor_SMD:C_0402_1005Metric
- C37: value 100nF -> 100nF/50V; footprint Capacitor_SMD:C_0603_1608Metric -> Capacitor_SMD:C_0402_1005Metric
- C38: value 100nF -> 22uF/16V; footprint Capacitor_SMD:C_0603_1608Metric -> Capacitor_SMD:C_0805_2012Metric
- C39: value 100nF -> 10uF/16V
- C40: value 100nF/50V -> 2.2uF/16V; footprint Capacitor_SMD:C_0603_1608Metric -> Capacitor_SMD:C_0402_1005Metric
- L1: value 22uH -> 6.8uH
- R1, R11, R2: footprint Resistor_SMD:R_0603_1608Metric -> Resistor_SMD:R_0402_1005Metric
- R10: value 10kΩ -> 0Ω; footprint Resistor_SMD:R_0603_1608Metric -> Resistor_SMD:R_0402_1005Metric
- R12: value 10kΩ -> 2.87kΩ(1%); footprint Resistor_SMD:R_0603_1608Metric -> Resistor_SMD:R_0402_1005Metric
- R13: value 470Ω -> 10kΩ; footprint Resistor_SMD:R_0603_1608Metric -> Resistor_SMD:R_0402_1005Metric
- R14: value 470Ω -> 510Ω; footprint Resistor_SMD:R_0603_1608Metric -> Resistor_SMD:R_0402_1005Metric
- R15: value 10kΩ -> 510Ω; footprint Resistor_SMD:R_0603_1608Metric -> Resistor_SMD:R_0402_1005Metric
- R16: value 0Ω -> 10kΩ; footprint Resistor_SMD:R_0603_1608Metric -> Resistor_SMD:R_0402_1005Metric
- R17: value 0Ω -> 100kΩ(1%); footprint Resistor_SMD:R_0603_1608Metric -> Resistor_SMD:R_0402_1005Metric
- R18: value 510Ω -> 33kΩ(1%); footprint Resistor_SMD:R_0603_1608Metric -> Resistor_SMD:R_0402_1005Metric
- R19: value 510Ω -> 100kΩ(1%); footprint Resistor_SMD:R_0603_1608Metric -> Resistor_SMD:R_0402_1005Metric
- R20: value 33Ω -> 18.7kΩ(1%); footprint Resistor_SMD:R_0603_1608Metric -> Resistor_SMD:R_0402_1005Metric
- R21, R22, R28, R29: value 33Ω -> 0Ω; footprint Resistor_SMD:R_0603_1608Metric -> Resistor_SMD:R_0402_1005Metric
- R23: value 33Ω -> 10kΩ(1%); footprint Resistor_SMD:R_0603_1608Metric -> Resistor_SMD:R_0402_1005Metric
- R24: value 510Ω -> 10kΩ; footprint Resistor_SMD:R_0603_1608Metric -> Resistor_SMD:R_0402_1005Metric
- R25: value 510Ω -> 470Ω; footprint Resistor_SMD:R_0603_1608Metric -> Resistor_SMD:R_0402_1005Metric
- R26: value 33Ω -> 470Ω; footprint Resistor_SMD:R_0603_1608Metric -> Resistor_SMD:R_0402_1005Metric
- R27: value 33Ω -> 10kΩ; footprint Resistor_SMD:R_0603_1608Metric -> Resistor_SMD:R_0402_1005Metric
- R3: value 10kΩ -> 5.1kΩ; footprint Resistor_SMD:R_0603_1608Metric -> Resistor_SMD:R_0402_1005Metric
- R32, R33: value 10kΩ -> 33Ω; footprint Resistor_SMD:R_0603_1608Metric -> Resistor_SMD:R_0402_1005Metric
- R35: value 47kΩ -> 510Ω; footprint Resistor_SMD:R_0603_1608Metric -> Resistor_SMD:R_0402_1005Metric
- R36: value 47kΩ -> 33Ω; footprint Resistor_SMD:R_0603_1608Metric -> Resistor_SMD:R_0402_1005Metric
- R4: value 100kΩ(1%) -> 5.1kΩ; footprint Resistor_SMD:R_0603_1608Metric -> Resistor_SMD:R_0402_1005Metric
- R5: value 33kΩ(1%) -> 10kΩ; footprint Resistor_SMD:R_0603_1608Metric -> Resistor_SMD:R_0402_1005Metric
- R6: value 2.87kΩ(1%) -> 10kΩ; footprint Resistor_SMD:R_0603_1608Metric -> Resistor_SMD:R_0402_1005Metric
- R7: value 13.7kΩ(1%) -> 10kΩ; footprint Resistor_SMD:R_0603_1608Metric -> Resistor_SMD:R_0402_1005Metric
- R8: value 10kΩ -> 330Ω; footprint Resistor_SMD:R_0603_1608Metric -> Resistor_SMD:R_0402_1005Metric
- R9: value 100kΩ(1%) -> 0Ω; footprint Resistor_SMD:R_0603_1608Metric -> Resistor_SMD:R_0402_1005Metric
- SHUNT1, SHUNT2: value 33mΩ -> 50mΩ; footprint Resistor_SMD:R_1206_3216Metric -> Resistor_SMD:R_0805_2012Metric
- TPA1, TPA2: footprint TestPoint:TestPoint_THTPad_2.0x2.0mm_Drill1.0mm -> TestPoint:TestPoint_THTPad_D2.0mm_Drill1.0mm
- U1: value TEENSY 4.0 -> USBLC6-2SC6; footprint SAVITAR:MODULE_DEV-15583 -> Package_TO_SOT_SMD:SOT-23-6
- U2: value ESP32-C3-MINI-1-H4X -> FSUSB42MUX; footprint SAVITAR:ESP32C3MINI1H4X -> SAVITAR:SOP50P490X110-10N
- U3: value TLV75733PDBV -> ATSAMD51J19A-A; footprint Package_TO_SOT_SMD:SOT-23-5 -> Package_QFP:TQFP-64_10x10mm_P0.5mm
- U4: value QRE1113GR -> ESP32-C3-MINI-1-H4X; footprint OptoDevice:OnSemi_CASE100CY -> SAVITAR:ESP32C3MINI1H4X
- U5: value QRE1113GR -> TLV75733PDBV; footprint OptoDevice:OnSemi_CASE100CY -> Package_TO_SOT_SMD:SOT-23-5
- moved C25 179.4 mm to (213.1, 182.0), turned to 90 degrees
- moved C14 176.4 mm to (208.5, 177.1)
- moved C24 173.8 mm to (213.1, 189.2), turned to 90 degrees
- moved C22 173.1 mm to (206.6, 178.4), turned to 180 degrees
- moved C16 170.9 mm to (208.5, 178.4)
- moved C23 167.7 mm to (204.3, 193.0), turned to 180 degrees
- moved U5 163.7 mm to (109.5, 163.3)
- moved C13 163.4 mm to (196.9, 184.3)
- moved C31 155.9 mm to (95.2, 181.4)
- moved C38 155.1 mm to (95.2, 188.1)
- moved U12 151.0 mm to (124.9, 143.2)
- moved U13 151.0 mm to (124.9, 148.0)
- moved U16 151.0 mm to (132.1, 143.2)
- moved U9 151.0 mm to (117.7, 148.0)
- moved U17 151.0 mm to (132.1, 148.0)
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Connections:
- net /TEENSY4 ESP32/MOT_B1 renamed /SAMD51 ESP32/MOT_B1
- net /TEENSY4 ESP32/MOT_B2 renamed /SAMD51 ESP32/MOT_B2
- net /TEENSY4 ESP32/SENSE_IN_A1 renamed /SAMD51 ESP32/SENSE_IN_A1
- net /TEENSY4 ESP32/SENSE_IN_B1 renamed /SAMD51 ESP32/SENSE_IN_B1
- C10 pad 1: GND -> VBAT
- C10 pad 2: +5V -> GND
- C12 pad 1: VBAT -> Net-(U3-PA00)
- C13 pad 1: GND -> Net-(U3-PA01)
- C13 pad 2: +5V -> GND
- C14 pad 1: VBAT -> Net-(U3-VDDCORE)
- C15 pad 1: +5V -> GND
- C15 pad 2: GND -> Net-(U3-~{RESET})
- C16 pad 1: Net-(IC1-SW) -> Net-(U3-VDDCORE)
- C16 pad 2: Net-(IC1-BS) -> GND
- C17 pad 1: +5V -> VBAT
- C17 pad 2: GND -> Net-(DRV2-VCP)
- C18 pad 2: VCC -> VBAT
- C19 pad 1: GND -> Net-(DRV2-CPH)
- C19 pad 2: +5V -> Net-(DRV2-CPL)
- C20 pad 1: GND -> VBAT
- C20 pad 2: /TEENSY4 ESP32/ESP_EN -> GND
- C21 pad 2: Net-(DRV2-VCP) -> GND
- C22 pad 1: VCC -> GND
- C22 pad 2: GND -> VCC
- C23 pad 2: VBAT -> VCC
- C24 pad 1: Net-(DRV2-CPH) -> GND
- C24 pad 2: Net-(DRV2-CPL) -> VCC
- C25 pad 1: VBAT -> GND
- C25 pad 2: GND -> VCC
- C27 pad 1: VBAT -> VCC
- C30 pad 1: GND -> Net-(IC1-SW)
- C30 pad 2: VCC -> Net-(IC1-BS)
- C31 pad 1: VCC -> VBAT
- C32 pad 1: VCC -> GND
- C32 pad 2: GND -> VCC
- C37 pad 1: VCC -> GND
- C37 pad 2: GND -> +3V8
- C39 pad 1: VCC -> GND
- C39 pad 2: GND -> +3V8
- C40 pad 1: VCC -> GND
- C40 pad 2: GND -> VCC
- DRV1 pad 1: /TEENSY4 ESP32/MOT_A.EN/IN1 -> /SAMD51 ESP32/MOT_A.EN/IN1
- DRV1 pad 10: /TEENSY4 ESP32/MOT_A2 -> /SAMD51 ESP32/MOT_A2
- DRV1 pad 16: /TEENSY4 ESP32/MOT_A.PMODE -> /SAMD51 ESP32/MOT_A.PMODE
- DRV1 pad 2: /TEENSY4 ESP32/MOT_A.PH/IN2 -> /SAMD51 ESP32/MOT_A.PH/IN2
- DRV1 pad 3: /TEENSY4 ESP32/MOT_A.~{SLEEP} -> /SAMD51 ESP32/MOT_A.~{SLEEP}
- DRV1 pad 4: /TEENSY4 ESP32/MOT_A.~{FAULT} -> /SAMD51 ESP32/MOT_A.~{FAULT}
- DRV1 pad 6: /TEENSY4 ESP32/MOT_A.C_STALL -> /SAMD51 ESP32/MOT_A.C_STALL
- DRV2 pad 1: /TEENSY4 ESP32/MOT_B.EN/IN1 -> /SAMD51 ESP32/MOT_B.EN/IN1
- DRV2 pad 16: /TEENSY4 ESP32/MOT_B.PMODE -> /SAMD51 ESP32/MOT_B.PMODE
- DRV2 pad 2: /TEENSY4 ESP32/MOT_B.PH/IN2 -> /SAMD51 ESP32/MOT_B.PH/IN2
- DRV2 pad 3: /TEENSY4 ESP32/MOT_B.~{SLEEP} -> /SAMD51 ESP32/MOT_B.~{SLEEP}
- DRV2 pad 4: /TEENSY4 ESP32/MOT_B.~{FAULT} -> /SAMD51 ESP32/MOT_B.~{FAULT}
- DRV2 pad 6: /TEENSY4 ESP32/MOT_B.C_STALL -> /SAMD51 ESP32/MOT_B.C_STALL
- INAA1 pad 1: /TEENSY4 ESP32/MOT_A1 -> /SAMD51 ESP32/MOT_A1
- INAA1 pad 5: /TEENSY4 ESP32/MOT_A.C_SENSE -> /SAMD51 ESP32/MOT_A.C_SENSE
- INAB1 pad 5: /TEENSY4 ESP32/MOT_B.C_SENSE -> /SAMD51 ESP32/MOT_B.C_SENSE
- J1 pad 1: /TEENSY4 ESP32/SEN_S0 -> /SAMD51 ESP32/SEN_S0
- J1 pad 2: /TEENSY4 ESP32/SEN_S1 -> /SAMD51 ESP32/SEN_S1
- J1 pad 3: /TEENSY4 ESP32/SEN_S2 -> /SAMD51 ESP32/SEN_S2
- J1 pad 4: /TEENSY4 ESP32/SEN_MUX1 -> /SAMD51 ESP32/SEN_MUX1
- J1 pad 5: /TEENSY4 ESP32/SEN_MUX2 -> /SAMD51 ESP32/SEN_MUX2
- J1 pad 6: /TEENSY4 ESP32/SEN_EN -> /SAMD51 ESP32/SEN_EN
- L1 pad 2: +5V -> +3V8
- MUX1 pad 1: /SENSOR ARRAY/S4 -> /SENSOR ARRAY/S11
- MUX1 pad 12: /SENSOR ARRAY/S3 -> /SENSOR ARRAY/S12
- MUX1 pad 13: /SENSOR ARRAY/S0 -> /SENSOR ARRAY/S15
- MUX1 pad 14: /SENSOR ARRAY/S1 -> /SENSOR ARRAY/S14
- MUX1 pad 15: /SENSOR ARRAY/S2 -> /SENSOR ARRAY/S13
- MUX1 pad 2: /SENSOR ARRAY/S6 -> /SENSOR ARRAY/S9
- MUX1 pad 3: /SENSOR ARRAY/COUT1 -> /SENSOR ARRAY/COUT2
- MUX1 pad 4: /SENSOR ARRAY/S7 -> /SENSOR ARRAY/S8
- MUX1 pad 5: /SENSOR ARRAY/S5 -> /SENSOR ARRAY/S10
- MUX2 pad 1: /SENSOR ARRAY/S11 -> /SENSOR ARRAY/S4
- MUX2 pad 12: /SENSOR ARRAY/S12 -> /SENSOR ARRAY/S3
- MUX2 pad 13: /SENSOR ARRAY/S15 -> /SENSOR ARRAY/S0
- MUX2 pad 14: /SENSOR ARRAY/S14 -> /SENSOR ARRAY/S1
- MUX2 pad 15: /SENSOR ARRAY/S13 -> /SENSOR ARRAY/S2
- MUX2 pad 2: /SENSOR ARRAY/S9 -> /SENSOR ARRAY/S6
- MUX2 pad 3: /SENSOR ARRAY/COUT2 -> /SENSOR ARRAY/COUT1
- MUX2 pad 4: /SENSOR ARRAY/S8 -> /SENSOR ARRAY/S7
- MUX2 pad 5: /SENSOR ARRAY/S10 -> /SENSOR ARRAY/S5
- R1 pad 1: /TEENSY4 ESP32/MOT_A.C_STALL -> /SAMD51 ESP32/MOT_A.C_STALL
- R10 pad 1: VCC -> /SAMD51 ESP32/SAMD_D+
- R10 pad 2: /TEENSY4 ESP32/MOT_B.PMODE -> Net-(U3-PA25)
- R11 pad 2: /TEENSY4 ESP32/ESP_EN -> Net-(U3-~{RESET})
- R12 pad 1: VCC -> /SAMD51 ESP32/MOT_B.C_STALL
- R12 pad 2: /TEENSY4 ESP32/ESP_BOOT -> GND
- R13 pad 1: /TEENSY4 ESP32/TNS_TX1 -> VCC
- R13 pad 2: Net-(R13-Pad2) -> /SAMD51 ESP32/MOT_B.~{FAULT}
- R14 pad 1: /TEENSY4 ESP32/TNS_RX1 -> /SAMD51 ESP32/STATUS_LED
- R14 pad 2: Net-(R14-Pad2) -> Net-(D1-A)
- R15 pad 1: VCC -> /SAMD51 ESP32/STATUS_LED
- R15 pad 2: Net-(U2-IO8) -> Net-(D2-A)
- R16 pad 1: Net-(R13-Pad2) -> VCC
- R16 pad 2: Net-(U2-RXD0) -> /SAMD51 ESP32/MOT_B.PMODE
- R17 pad 1: Net-(R14-Pad2) -> /SAMD51 ESP32/BAT_LEVEL
- R17 pad 2: Net-(U2-TXD0) -> VBAT
- R18 pad 1: /TEENSY4 ESP32/STATUS_LED -> GND
- R18 pad 2: Net-(D1-A) -> /SAMD51 ESP32/BAT_LEVEL
- R19 pad 1: /TEENSY4 ESP32/STATUS_LED -> +3V8
- R19 pad 2: Net-(D2-A) -> Net-(IC1-FB)
- R2 pad 2: /TEENSY4 ESP32/MOT_A.~{FAULT} -> /SAMD51 ESP32/MOT_A.~{FAULT}
- R20 pad 1: Net-(U5-A) -> Net-(IC1-FB)
- R20 pad 2: Net-(U4-K) -> GND
- R21 pad 1: Net-(U7-A) -> /SAMD51 ESP32/ESP_D-
- R21 pad 2: Net-(U6-K) -> Net-(U4-IO18)
- R22 pad 1: Net-(U9-A) -> /SAMD51 ESP32/ESP_D+
- R22 pad 2: Net-(U8-K) -> Net-(U4-IO19)
- R23 pad 1: Net-(U11-A) -> VCC
- R23 pad 2: Net-(U10-K) -> /SAMD51 ESP32/ESP_EN
- R24 pad 1: /SENSOR ARRAY/EN -> VCC
- R24 pad 2: Net-(D3-A) -> /SAMD51 ESP32/ESP_BOOT
- R25 pad 1: /SENSOR ARRAY/EN -> /SAMD51 ESP32/SAMD_TX1
- R25 pad 2: Net-(D4-A) -> Net-(R25-Pad2)
- R26 pad 1: Net-(U13-A) -> /SAMD51 ESP32/SAMD_RX1
- R26 pad 2: Net-(U12-K) -> Net-(R26-Pad2)
- R27 pad 1: Net-(U15-A) -> VCC
- R27 pad 2: Net-(U14-K) -> Net-(U4-IO8)
- R28 pad 1: Net-(U17-A) -> Net-(R25-Pad2)
- R28 pad 2: Net-(U16-K) -> Net-(U4-RXD0)
- R29 pad 1: Net-(U19-A) -> Net-(R26-Pad2)
- R29 pad 2: Net-(U18-K) -> Net-(U4-TXD0)
- R3 pad 1: VCC -> GND
- R3 pad 2: /TEENSY4 ESP32/MOT_A.PMODE -> Net-(USBC1-CC1)
- R32 pad 1: /SENSOR ARRAY/EN -> Net-(U11-A)
- R32 pad 2: Net-(Q1-B) -> Net-(U10-K)
- R33 pad 1: /SENSOR ARRAY/~{EN} -> Net-(U13-A)
- R33 pad 2: VCC -> Net-(U12-K)
- R35 pad 1: /SENSOR ARRAY/COUT2 -> /SENSOR ARRAY/EN
- R35 pad 2: VCC -> Net-(D4-A)
- R36 pad 1: /SENSOR ARRAY/COUT1 -> Net-(U15-A)
- R36 pad 2: VCC -> Net-(U14-K)
- R4 pad 1: /TEENSY4 ESP32/BAT_LEVEL -> GND
- R4 pad 2: VBAT -> Net-(USBC1-CC2)
- R5 pad 1: GND -> VCC
- R5 pad 2: /TEENSY4 ESP32/BAT_LEVEL -> /SAMD51 ESP32/MOT_A.PMODE
- R6 pad 1: /TEENSY4 ESP32/MOT_B.C_STALL -> VCC
- R6 pad 2: GND -> /SAMD51 ESP32/SWCLK
- R7 pad 1: Net-(IC1-FB) -> Net-(U2-/OE)
- R8 pad 1: VCC -> Net-(R8-Pad1)
- R8 pad 2: /TEENSY4 ESP32/MOT_B.~{FAULT} -> Net-(U3-~{RESET})
- R9 pad 1: Net-(IC1-FB) -> /SAMD51 ESP32/SAMD_D-
- R9 pad 2: +5V -> Net-(U3-PA24)
- SHUNT2 pad 1: /TEENSY4 ESP32/MOT_A1 -> /SAMD51 ESP32/MOT_A1
- TPA1 pad 1: /TEENSY4 ESP32/MOT_A1 -> /SAMD51 ESP32/SWCLK
- TPA2 pad 1: /TEENSY4 ESP32/MOT_A2 -> /SAMD51 ESP32/SWDIO
- U1 pad 1: /TEENSY4 ESP32/TNS_TX1 -> Net-(U1-I/O1-Pad1)
- U1 pad 2: /TEENSY4 ESP32/MOT_A.EN/IN1 -> GND
- U1 pad 3: /TEENSY4 ESP32/MOT_A.PH/IN2 -> Net-(U1-I/O2-Pad3)
- U1 pad 4: /TEENSY4 ESP32/MOT_A.~{SLEEP} -> /SAMD51 ESP32/D+
- U1 pad 5: /TEENSY4 ESP32/MOT_A.~{FAULT} -> VBUS
- U1 pad 6: /TEENSY4 ESP32/MOT_A.PMODE -> /SAMD51 ESP32/D-
- U10 pad 3: /SENSOR ARRAY/S3 -> /SENSOR ARRAY/S2
- U11 pad 2: /SENSOR ARRAY/3_12_LED -> /SENSOR ARRAY/2_13_LED
- U11 pad 3: /SENSOR ARRAY/S12 -> /SENSOR ARRAY/S13
- U12 pad 3: /SENSOR ARRAY/S4 -> /SENSOR ARRAY/S3
- U13 pad 2: /SENSOR ARRAY/4_11_LED -> /SENSOR ARRAY/3_12_LED
- U13 pad 3: /SENSOR ARRAY/S11 -> /SENSOR ARRAY/S12
- U14 pad 3: /SENSOR ARRAY/S5 -> /SENSOR ARRAY/S4
- U15 pad 2: /SENSOR ARRAY/5_10_LED -> /SENSOR ARRAY/4_11_LED
- U15 pad 3: /SENSOR ARRAY/S10 -> /SENSOR ARRAY/S11
- U16 pad 3: /SENSOR ARRAY/S6 -> /SENSOR ARRAY/S5
- U17 pad 2: /SENSOR ARRAY/6_9_LED -> /SENSOR ARRAY/5_10_LED
- U17 pad 3: /SENSOR ARRAY/S9 -> /SENSOR ARRAY/S10
- U18 pad 3: /SENSOR ARRAY/S7 -> /SENSOR ARRAY/S6
- U19 pad 2: /SENSOR ARRAY/7_8_LED -> /SENSOR ARRAY/6_9_LED
- U19 pad 3: /SENSOR ARRAY/S8 -> /SENSOR ARRAY/S9
- U2 pad 1: GND -> VCC
- U2 pad 10: unconnected-(U2-NC_4-Pad10) -> Net-(U2-/OE)
- U2 pad 2: GND -> /SAMD51 ESP32/USB_SEL
- U2 pad 3: VCC -> /SAMD51 ESP32/D+
- U2 pad 4: unconnected-(U2-NC_1-Pad4) -> /SAMD51 ESP32/D-
- U2 pad 5: unconnected-(U2-IO2-Pad5) -> GND
- U2 pad 6: unconnected-(U2-IO3-Pad6) -> /SAMD51 ESP32/ESP_D-
- U2 pad 7: unconnected-(U2-NC_2-Pad7) -> /SAMD51 ESP32/ESP_D+
- U2 pad 8: /TEENSY4 ESP32/ESP_EN -> /SAMD51 ESP32/SAMD_D-
- U2 pad 9: unconnected-(U2-NC_3-Pad9) -> /SAMD51 ESP32/SAMD_D+
- U3 pad 1: +5V -> Net-(U3-PA00)
- U3 pad 2: GND -> Net-(U3-PA01)
- U3 pad 3: +5V -> unconnected-(U3-PA02-Pad3)
- U3 pad 5: VCC -> unconnected-(U3-PB04-Pad5)
- U4 pad 1: VCC -> GND
- U4 pad 2: Net-(U4-K) -> GND
- U4 pad 3: /SENSOR ARRAY/S0 -> VCC
- U4 pad 4: GND -> unconnected-(U4-NC_1-Pad4)
- U5 pad 1: Net-(U5-A) -> +3V8
- U5 pad 2: /SENSOR ARRAY/0_15_LED -> GND
- U5 pad 3: /SENSOR ARRAY/S15 -> +3V8
- U5 pad 4: GND -> unconnected-(U5-NC-Pad4)
- U6 pad 3: /SENSOR ARRAY/S1 -> /SENSOR ARRAY/S0
- U7 pad 2: /SENSOR ARRAY/1_14_LED -> /SENSOR ARRAY/0_15_LED
- U7 pad 3: /SENSOR ARRAY/S14 -> /SENSOR ARRAY/S15
- U8 pad 3: /SENSOR ARRAY/S2 -> /SENSOR ARRAY/S1
- U9 pad 2: /SENSOR ARRAY/2_13_LED -> /SENSOR ARRAY/1_14_LED
- U9 pad 3: /SENSOR ARRAY/S13 -> /SENSOR ARRAY/S14
Other:
- outline, holes or cut-outs redrawn
- copper layers 2 -> 4
