File: SAVITAR_V2.kicad_pcb (KiCad board)
At the start: 4 copper layers, 127.2 x 119.8 mm, 148 parts, among them IC1 MT2492, J1 FH34SRJ-8S-0.5SH_50_, J2 FH34SRJ-8S-0.5SH_50_, Q1 MMBT3904, SW1 TS-1088-AR02016, SW2 TS-1088-AR02016, SW3 TS-1088-AR02016, U1 USBLC6-2SC6, U10 QRE1113GR, U11 QRE1113GR, U12 QRE1113GR, U13 QRE1113GR, U14 QRE1113GR, U15 QRE1113GR, U16 QRE1113GR, U17 QRE1113GR, U18 QRE1113GR, U19 QRE1113GR, U2 FSUSB42MUX, U20 QRE1113GR, U21 QRE1113GR, U3 ATSAMD51J19A-A, U4 ESP32-C3-MINI-1-H4X, U5 TLV75733PDBV, U6 QRE1113GR, U7 QRE1113GR, U8 QRE1113GR, U9 QRE1113GR, Y1 32.768kHz

Commit message: Will add info in a later commit
Parts:
- removed C34: 22uF/16V, LED_SMD:LED_0805_2012Metric
- removed C35, C38: 22uF/16V, Capacitor_SMD:C_0805_2012Metric
- removed C36, C42: 1uF/16V, Capacitor_SMD:C_0402_1005Metric
- removed C37, C41, C46, C49: 100nF/50V, Capacitor_SMD:C_0402_1005Metric
- removed C39: 10uF/16V, Capacitor_SMD:C_0603_1608Metric
- removed C40: 2.2uF/16V, Capacitor_SMD:C_0402_1005Metric
- removed C43, C44, C45: 100nF, Capacitor_SMD:C_0402_1005Metric
- removed C47, C48: 100uF/25V, Capacitor_SMD:CP_Elec_6.3x5.8
- removed INAA1, INAB1: INA240A1DR, SAVITAR:SOIC127P600X175-8N
- removed R41, R43: 10kΩ, Resistor_SMD:R_0402_1005Metric
- removed R42: 47kΩ, Resistor_SMD:R_0402_1005Metric
- removed S1: SSSS811101, SAVITAR:SSSS811101
- removed SHUNT1, SHUNT2: 50mΩ, Resistor_SMD:R_0805_2012Metric
- removed SW2, SW3: TS-1088-AR02016, Button_Switch_SMD:SW_SPST_TS-1088-xR020
- removed TPA3, TPA4, TPA5: TestPoint, TestPoint:TestPoint_THTPad_D2.0mm_Drill1.0mm
- removed TPA6, TPA7: TestPoint, TestPoint:TestPoint_THTPad_2.0x2.0mm_Drill1.0mm
- removed U21: QRE1113GR, OptoDevice:OnSemi_CASE100CY
- removed Y1: 32.768kHz, Crystal:Crystal_SMD_3215-2Pin_3.2x1.5mm
- added C26: 10uF/16V, Capacitor_SMD:C_0603_1608Metric, F.Cu at (202.4, 187.8)
- added SWD_CLK1: TestPoint, TestPoint:TestPoint_THTPad_D2.0mm_Drill1.0mm, F.Cu at (165.3, 172.8)
- added SWD_GND1: TestPoint, TestPoint:TestPoint_THTPad_D2.0mm_Drill1.0mm, F.Cu at (169.4, 172.8)
- added SWD_IO1: TestPoint, TestPoint:TestPoint_THTPad_D2.0mm_Drill1.0mm, F.Cu at (163.4, 169.8)
- added SWD_PWR1: TestPoint, TestPoint:TestPoint_THTPad_D2.0mm_Drill1.0mm, F.Cu at (167.4, 169.8)
- added SWD_RST1: TestPoint, TestPoint:TestPoint_THTPad_D2.0mm_Drill1.0mm, F.Cu at (171.5, 169.8)
- added TP1: TestPoint, TestPoint:TestPoint_THTPad_D2.0mm_Drill1.0mm, F.Cu at (212.4, 170.8)
- added TP2: TestPoint, TestPoint:TestPoint_THTPad_D2.0mm_Drill1.0mm, F.Cu at (209.4, 170.8)
- C1: value 100nF/50V -> 10uF (X7R); footprint Capacitor_SMD:C_0402_1005Metric -> Capacitor_SMD:C_0603_1608Metric
- C10, C9: value 47uF -> 100nF; footprint Capacitor_SMD:C_1206_3216Metric -> Capacitor_SMD:C_0402_1005Metric
- C11, C31: value 47uF/25V -> 100nF; footprint Capacitor_SMD:C_1206_3216Metric -> Capacitor_SMD:C_0402_1005Metric
- C12: value 18pF/25V -> 22uF/16V; footprint Capacitor_SMD:C_0402_1005Metric -> Capacitor_SMD:C_0805_2012Metric
- C13: value 18pF/25V -> 100nF/16V
- C14: value 10uF (X7R) -> 100nF/50V; footprint Capacitor_SMD:C_0603_1608Metric -> Capacitor_SMD:C_0402_1005Metric
- C15: value 1uF/16V -> 22nF/50V; footprint Capacitor_SMD:C_0603_1608Metric -> Capacitor_SMD:C_0402_1005Metric
- C16: value 1uF (X7R) -> 22uF/25V; footprint Capacitor_SMD:C_0402_1005Metric -> Capacitor_SMD:C_0805_2012Metric
- C17: value 100nF/16V -> 100uF/25V; footprint Capacitor_SMD:C_0402_1005Metric -> Capacitor_SMD:CP_Elec_6.3x5.8
- C2: value 100nF/50V -> 100nF/16V
- C20: value 22uF/25V -> 22uF/16V
- C21, C29: value 47uF -> 1uF/16V; footprint Capacitor_SMD:C_1206_3216Metric -> Capacitor_SMD:C_0402_1005Metric
- C22: value 100nF (X7R) -> 22pF; footprint Capacitor_SMD:C_0402_1005Metric -> Capacitor_SMD:C_0603_1608Metric
- C23: value 100nF -> 22uF/16V; footprint Capacitor_SMD:C_0402_1005Metric -> Capacitor_SMD:C_0805_2012Metric
- C24: value 100nF -> 22uF/16V; footprint Capacitor_SMD:C_0402_1005Metric -> LED_SMD:LED_0805_2012Metric
- C25: value 100nF -> 100nF/50V
- C27: value 22uF/16V -> 2.2uF/16V; footprint Capacitor_SMD:C_0805_2012Metric -> Capacitor_SMD:C_0402_1005Metric
- C28: value 47uF -> 100nF/50V; footprint Capacitor_SMD:C_1206_3216Metric -> Capacitor_SMD:C_0402_1005Metric
- C3: value 2.2uF/16V -> 100nF/50V
- C30: value 22nF/50V -> 100nF
- C32: value 100nF/50V -> 100nF
- C33: value 22pF -> 100nF/50V; footprint Capacitor_SMD:C_0603_1608Metric -> Capacitor_SMD:C_0402_1005Metric
- C4: value 2.2uF/16V -> 22nF/50V
- C5: value 100nF/16V -> 1uF (X7R)
- C6: value 100nF/50V -> 100uF/25V; footprint Capacitor_SMD:C_0402_1005Metric -> Capacitor_SMD:CP_Elec_6.3x5.8
- C7: value 22nF/50V -> 100nF/50V
- C8: value 47uF -> 100nF (X7R); footprint Capacitor_SMD:C_1206_3216Metric -> Capacitor_SMD:C_0402_1005Metric
- R10: value 0Ω -> 510Ω
- R11: value 10kΩ(1%) -> 510Ω
- R12: value 2.87kΩ(1%) -> 10kΩ
- R13: value 10kΩ -> 100kΩ(1%)
- R14: value 510Ω -> 33kΩ(1%)
- R15: value 510Ω -> 0Ω
- R16: value 10kΩ -> 0Ω
- R17: value 100kΩ(1%) -> 10kΩ(1%)
- R18: value 33kΩ(1%) -> 100kΩ(1%)
- R19: value 100kΩ(1%) -> 18.7kΩ(1%)
- R20: value 18.7kΩ(1%) -> 10kΩ
- R21, R22: value 0Ω -> 470Ω
- R23: value 10kΩ(1%) -> 10kΩ
- R25, R26: value 470Ω -> 0Ω
- R27: value 10kΩ -> 33Ω
- R28, R29: value 0Ω -> 33Ω
- R3, R4: value 5.1kΩ -> 10kΩ
- R31, R32: value 33Ω -> 510Ω
- R34, R35: value 510Ω -> 33Ω
- R37, R39: value 33Ω -> 47kΩ
- R38: value 33Ω -> 10kΩ
- R40: value 47kΩ -> 10kΩ
- R5: value 10kΩ -> 10kΩ(1%)
- R6, R7: value 10kΩ -> 5.1kΩ
- R8: value 330Ω -> 2.87kΩ(1%)
- R9: value 0Ω -> 10kΩ
- TPA1, TPA2: footprint TestPoint:TestPoint_THTPad_D2.0mm_Drill1.0mm -> TestPoint:TestPoint_THTPad_2.0x2.0mm_Drill1.0mm
- U2: value FSUSB42MUX -> ATSAMD51J19A-A; footprint SAVITAR:SOP50P490X110-10N -> Package_QFP:TQFP-64_10x10mm_P0.5mm
- U3: value ATSAMD51J19A-A -> ESP32-C3-MINI-1-H4X; footprint Package_QFP:TQFP-64_10x10mm_P0.5mm -> SAVITAR:ESP32C3MINI1H4X
- U4: value ESP32-C3-MINI-1-H4X -> TLV75733PDBV; footprint SAVITAR:ESP32C3MINI1H4X -> Package_TO_SOT_SMD:SOT-23-5
- U5: value TLV75733PDBV -> QRE1113GR; footprint Package_TO_SOT_SMD:SOT-23-5 -> OptoDevice:OnSemi_CASE100CY
- moved R13 223.5 mm to (317.2, 118.2)
- moved R14 223.5 mm to (317.2, 120.7)
- moved R18 223.5 mm to (317.2, 130.7)
- moved R19 223.5 mm to (317.2, 133.2)
- moved D3 177.6 mm to (144.1, -45.1)
- moved D4 177.6 mm to (144.1, -42.6)
- moved DEMUX1 177.6 mm to (119.7, -10.3)
- moved J2 177.6 mm to (134.6, -11.1)
- moved MUX1 177.6 mm to (117.4, -21.2)
- moved MUX2 177.6 mm to (125.9, -21.2)
- moved R31 177.6 mm to (136.1, -20.9)
- moved R36 177.6 mm to (140.1, -20.9)
- moved U11 177.6 mm to (124.0, -39.2)
- moved U15 177.6 mm to (131.2, -39.2)
- moved U19 177.6 mm to (138.4, -39.2)
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Connections:
- C1 pad 1: GND -> Net-(U2-VDDCORE)
- C1 pad 2: VCC -> GND
- C10 pad 1: VBAT -> GND
- C10 pad 2: GND -> VCC
- C11 pad 1: VBAT -> GND
- C11 pad 2: GND -> VCC
- C12 pad 1: Net-(U3-PA00) -> VCC
- C13 pad 1: Net-(U3-PA01) -> VBAT
- C13 pad 2: GND -> Net-(DRV2-VCP)
- C14 pad 1: Net-(U3-VDDCORE) -> GND
- C14 pad 2: GND -> VBAT
- C15 pad 1: GND -> Net-(DRV2-CPH)
- C15 pad 2: Net-(U3-~{RESET}) -> Net-(DRV2-CPL)
- C16 pad 1: Net-(U3-VDDCORE) -> VBAT
- C17 pad 2: Net-(DRV2-VCP) -> GND
- C18 pad 2: VBAT -> VCC
- C19 pad 1: Net-(DRV2-CPH) -> Net-(IC1-SW)
- C19 pad 2: Net-(DRV2-CPL) -> Net-(IC1-BS)
- C2 pad 1: GND -> VBAT
- C2 pad 2: VCC -> Net-(DRV1-VCP)
- C20 pad 1: VBAT -> VCC
- C21 pad 1: VBAT -> GND
- C21 pad 2: GND -> /SAMD51 ESP32/ESP_EN
- C22 pad 1: GND -> Net-(IC1-FB)
- C22 pad 2: VCC -> +3V8
- C23 pad 1: GND -> VCC
- C23 pad 2: VCC -> GND
- C24 pad 1: GND -> +3V8
- C24 pad 2: VCC -> GND
- C25 pad 2: VCC -> +3V8
- C27 pad 1: VCC -> GND
- C27 pad 2: GND -> VCC
- C28 pad 1: VBAT -> VCC
- C29 pad 1: VBAT -> VCC
- C3 pad 2: VCC -> VBAT
- C30 pad 1: Net-(IC1-SW) -> VCC
- C30 pad 2: Net-(IC1-BS) -> GND
- C31 pad 1: VBAT -> VCC
- C32 pad 1: GND -> VCC
- C32 pad 2: VCC -> GND
- C33 pad 1: Net-(IC1-FB) -> VCC
- C33 pad 2: +3V8 -> GND
- C4 pad 1: GND -> Net-(DRV1-CPH)
- C4 pad 2: VCC -> Net-(DRV1-CPL)
- C5 pad 1: VBAT -> Net-(U2-VDDCORE)
- C5 pad 2: Net-(DRV1-VCP) -> GND
- C6 pad 1: GND -> VBAT
- C6 pad 2: VBAT -> GND
- C7 pad 1: Net-(DRV1-CPH) -> /SAMD51 ESP32/SWD1
- C7 pad 2: Net-(DRV1-CPL) -> GND
- C8 pad 1: VBAT -> GND
- C8 pad 2: GND -> VCC
- C9 pad 1: VBAT -> GND
- C9 pad 2: GND -> VCC
- FB1 pad 2: Net-(U3-VDDANA) -> /SAMD51 ESP32/SWD1
- R10 pad 1: /SAMD51 ESP32/SAMD_D+ -> /SAMD51 ESP32/STATUS_LED
- R10 pad 2: Net-(U3-PA25) -> Net-(D1-A)
- R11 pad 1: VCC -> /SAMD51 ESP32/STATUS_LED
- R11 pad 2: Net-(U3-~{RESET}) -> Net-(D2-A)
- R12 pad 1: /SAMD51 ESP32/MOT_B.C_STALL -> VCC
- R12 pad 2: GND -> /SAMD51 ESP32/MOT_B.PMODE
- R13 pad 1: VCC -> /SAMD51 ESP32/BAT_LEVEL
- R13 pad 2: /SAMD51 ESP32/MOT_B.~{FAULT} -> VBAT
- R14 pad 1: /SAMD51 ESP32/STATUS_LED -> GND
- R14 pad 2: Net-(D1-A) -> /SAMD51 ESP32/BAT_LEVEL
- R15 pad 1: /SAMD51 ESP32/STATUS_LED -> /SAMD51 ESP32/ESP_D-
- R15 pad 2: Net-(D2-A) -> Net-(U3-IO18)
- R16 pad 1: VCC -> /SAMD51 ESP32/ESP_D+
- R16 pad 2: /SAMD51 ESP32/MOT_B.PMODE -> Net-(U3-IO19)
- R17 pad 1: /SAMD51 ESP32/BAT_LEVEL -> VCC
- R17 pad 2: VBAT -> /SAMD51 ESP32/ESP_EN
- R18 pad 1: GND -> +3V8
- R18 pad 2: /SAMD51 ESP32/BAT_LEVEL -> Net-(IC1-FB)
- R19 pad 1: +3V8 -> Net-(IC1-FB)
- R19 pad 2: Net-(IC1-FB) -> GND
- R20 pad 1: Net-(IC1-FB) -> VCC
- R20 pad 2: GND -> /SAMD51 ESP32/ESP_BOOT
- R21 pad 1: /SAMD51 ESP32/ESP_D- -> /SAMD51 ESP32/SAMD_TX1
- R21 pad 2: Net-(U4-IO18) -> Net-(R21-Pad2)
- R22 pad 1: /SAMD51 ESP32/ESP_D+ -> /SAMD51 ESP32/SAMD_RX1
- R22 pad 2: Net-(U4-IO19) -> Net-(R22-Pad2)
- R23 pad 2: /SAMD51 ESP32/ESP_EN -> Net-(U3-IO2)
- R24 pad 2: /SAMD51 ESP32/ESP_BOOT -> Net-(U3-IO8)
- R25 pad 1: /SAMD51 ESP32/SAMD_TX1 -> Net-(R21-Pad2)
- R25 pad 2: Net-(R25-Pad2) -> Net-(U3-RXD0)
- R26 pad 1: /SAMD51 ESP32/SAMD_RX1 -> Net-(R22-Pad2)
- R26 pad 2: Net-(R26-Pad2) -> Net-(U3-TXD0)
- R27 pad 1: VCC -> Net-(U6-A)
- R27 pad 2: Net-(U4-IO8) -> Net-(U5-K)
- R28 pad 1: Net-(R25-Pad2) -> Net-(U8-A)
- R28 pad 2: Net-(U4-RXD0) -> Net-(U7-K)
- R29 pad 1: Net-(R26-Pad2) -> Net-(U10-A)
- R29 pad 2: Net-(U4-TXD0) -> Net-(U9-K)
- R3 pad 1: GND -> VCC
- R3 pad 2: Net-(USBC1-CC1) -> /SAMD51 ESP32/MOT_A.PMODE
- R30 pad 1: Net-(U7-A) -> Net-(U12-A)
- R30 pad 2: Net-(U6-K) -> Net-(U11-K)
- R31 pad 1: Net-(U9-A) -> /SENSOR ARRAY/EN
- R31 pad 2: Net-(U8-K) -> Net-(D3-A)
- R32 pad 1: Net-(U11-A) -> /SENSOR ARRAY/EN
- R32 pad 2: Net-(U10-K) -> Net-(D4-A)
- R33 pad 1: Net-(U13-A) -> Net-(U14-A)
- R33 pad 2: Net-(U12-K) -> Net-(U13-K)
- R34 pad 1: /SENSOR ARRAY/EN -> Net-(U16-A)
- R34 pad 2: Net-(D3-A) -> Net-(U15-K)
- R35 pad 1: /SENSOR ARRAY/EN -> Net-(U18-A)
- R35 pad 2: Net-(D4-A) -> Net-(U17-K)
- R36 pad 1: Net-(U15-A) -> Net-(U20-A)
- R36 pad 2: Net-(U14-K) -> Net-(U19-K)
- R37 pad 1: Net-(U17-A) -> /SENSOR ARRAY/COUT2
- R37 pad 2: Net-(U16-K) -> VCC
- R38 pad 1: Net-(U19-A) -> /SENSOR ARRAY/EN
- R38 pad 2: Net-(U18-K) -> Net-(Q1-B)
- R39 pad 1: Net-(U21-A) -> /SENSOR ARRAY/COUT1
- R39 pad 2: Net-(U20-K) -> VCC
- R4 pad 1: GND -> VCC
- R4 pad 2: Net-(USBC1-CC2) -> /SAMD51 ESP32/SWCLK
- R40 pad 1: /SENSOR ARRAY/COUT2 -> /SENSOR ARRAY/~{EN}
- R5 pad 2: /SAMD51 ESP32/MOT_A.PMODE -> /SAMD51 ESP32/SWD5
- R6 pad 1: VCC -> GND
- R6 pad 2: /SAMD51 ESP32/SWCLK -> Net-(USBC1-CC1)
- R7 pad 1: Net-(U2-/OE) -> GND
- R7 pad 2: GND -> Net-(USBC1-CC2)
- R8 pad 1: Net-(R8-Pad1) -> /SAMD51 ESP32/MOT_B.C_STALL
- R8 pad 2: Net-(U3-~{RESET}) -> GND
- R9 pad 1: /SAMD51 ESP32/SAMD_D- -> VCC
- R9 pad 2: Net-(U3-PA24) -> /SAMD51 ESP32/MOT_B.~{FAULT}
- SW1 pad 2: Net-(R8-Pad1) -> /SAMD51 ESP32/SWD5
- TPA1 pad 1: /SAMD51 ESP32/SWCLK -> /SAMD51 ESP32/MOT_A1
- TPA2 pad 1: /SAMD51 ESP32/SWDIO -> /SAMD51 ESP32/MOT_A2
- U1 pad 4: /SAMD51 ESP32/D+ -> /SAMD51 ESP32/ESP_D+
- U1 pad 6: /SAMD51 ESP32/D- -> /SAMD51 ESP32/ESP_D-
- U10 pad 1: VCC -> Net-(U10-A)
- U10 pad 2: Net-(U10-K) -> /SENSOR ARRAY/2_13_LED
- U10 pad 3: /SENSOR ARRAY/S2 -> /SENSOR ARRAY/S13
- U11 pad 1: Net-(U11-A) -> VCC
- U11 pad 2: /SENSOR ARRAY/2_13_LED -> Net-(U11-K)
- U11 pad 3: /SENSOR ARRAY/S13 -> /SENSOR ARRAY/S3
- U12 pad 1: VCC -> Net-(U12-A)
- U12 pad 2: Net-(U12-K) -> /SENSOR ARRAY/3_12_LED
- U12 pad 3: /SENSOR ARRAY/S3 -> /SENSOR ARRAY/S12
- U13 pad 1: Net-(U13-A) -> VCC
- U13 pad 2: /SENSOR ARRAY/3_12_LED -> Net-(U13-K)
- U13 pad 3: /SENSOR ARRAY/S12 -> /SENSOR ARRAY/S4
- U14 pad 1: VCC -> Net-(U14-A)
- U14 pad 2: Net-(U14-K) -> /SENSOR ARRAY/4_11_LED
- U14 pad 3: /SENSOR ARRAY/S4 -> /SENSOR ARRAY/S11
- U15 pad 1: Net-(U15-A) -> VCC
- U15 pad 2: /SENSOR ARRAY/4_11_LED -> Net-(U15-K)
- U15 pad 3: /SENSOR ARRAY/S11 -> /SENSOR ARRAY/S5
- U16 pad 1: VCC -> Net-(U16-A)
- U16 pad 2: Net-(U16-K) -> /SENSOR ARRAY/5_10_LED
- U16 pad 3: /SENSOR ARRAY/S5 -> /SENSOR ARRAY/S10
- U17 pad 1: Net-(U17-A) -> VCC
- U17 pad 2: /SENSOR ARRAY/5_10_LED -> Net-(U17-K)
- U17 pad 3: /SENSOR ARRAY/S10 -> /SENSOR ARRAY/S6
- U18 pad 1: VCC -> Net-(U18-A)
- U18 pad 2: Net-(U18-K) -> /SENSOR ARRAY/6_9_LED
- U18 pad 3: /SENSOR ARRAY/S6 -> /SENSOR ARRAY/S9
- U19 pad 1: Net-(U19-A) -> VCC
- U19 pad 2: /SENSOR ARRAY/6_9_LED -> Net-(U19-K)
- U19 pad 3: /SENSOR ARRAY/S9 -> /SENSOR ARRAY/S7
- U2 pad 1: VCC -> unconnected-(U2-PA00-Pad1)
- U2 pad 10: Net-(U2-/OE) -> unconnected-(U2-PB07-Pad10)
- U2 pad 2: /SAMD51 ESP32/USB_SEL -> unconnected-(U2-PA01-Pad2)
- U2 pad 3: /SAMD51 ESP32/D+ -> unconnected-(U2-PA02-Pad3)
- U2 pad 4: /SAMD51 ESP32/D- -> unconnected-(U2-PA03-Pad4)
- U2 pad 5: GND -> unconnected-(U2-PB04-Pad5)
- U2 pad 6: /SAMD51 ESP32/ESP_D- -> unconnected-(U2-PB05-Pad6)
- U2 pad 7: /SAMD51 ESP32/ESP_D+ -> GND
- U2 pad 8: /SAMD51 ESP32/SAMD_D- -> /SAMD51 ESP32/SWD1
- U2 pad 9: /SAMD51 ESP32/SAMD_D+ -> unconnected-(U2-PB06-Pad9)
- U20 pad 1: VCC -> Net-(U20-A)
- U20 pad 2: Net-(U20-K) -> /SENSOR ARRAY/7_8_LED
- U20 pad 3: /SENSOR ARRAY/S7 -> /SENSOR ARRAY/S8
- U3 pad 1: Net-(U3-PA00) -> GND
- U3 pad 11: unconnected-(U3-PB08-Pad11) -> GND
- U3 pad 14: unconnected-(U3-PA05-Pad14) -> GND
- U3 pad 2: Net-(U3-PA01) -> GND
- U3 pad 21: VCC -> unconnected-(U3-IO7-Pad21)
- U3 pad 22: GND -> Net-(U3-IO8)
- U3 pad 23: unconnected-(U3-PB10-Pad23) -> /SAMD51 ESP32/ESP_BOOT
- U3 pad 26: unconnected-(U3-PB13-Pad26) -> Net-(U3-IO18)
- U3 pad 27: unconnected-(U3-PB14-Pad27) -> Net-(U3-IO19)
- U3 pad 3: unconnected-(U3-PA02-Pad3) -> VCC
- U3 pad 30: unconnected-(U3-PA13-Pad30) -> Net-(U3-RXD0)
- U3 pad 31: unconnected-(U3-PA14-Pad31) -> Net-(U3-TXD0)
- U3 pad 33: GND -> unconnected-(U3-NC_12-Pad33)
- U3 pad 34: VCC -> unconnected-(U3-NC_13-Pad34)
- U3 pad 36: unconnected-(U3-PA17-Pad36) -> GND
- U3 pad 37: unconnected-(U3-PA18-Pad37) -> GND
- U3 pad 38: unconnected-(U3-PA19-Pad38) -> GND
- U3 pad 39: unconnected-(U3-PB16-Pad39) -> GND
- U3 pad 40: unconnected-(U3-PB17-Pad40) -> GND
- U3 pad 41: unconnected-(U3-PA20-Pad41) -> GND
- U3 pad 42: unconnected-(U3-PA21-Pad42) -> GND
- U3 pad 43: unconnected-(U3-PA22-Pad43) -> GND
- U3 pad 44: unconnected-(U3-PA23-Pad44) -> GND
- U3 pad 45: Net-(U3-PA24) -> GND
- U3 pad 46: Net-(U3-PA25) -> GND
- U3 pad 48: VCC -> GND
- U3 pad 49: unconnected-(U3-PB22-Pad49) -> GND
- U3 pad 5: unconnected-(U3-PB04-Pad5) -> Net-(U3-IO2)
- U3 pad 50: unconnected-(U3-PB23-Pad50) -> GND
- U3 pad 51: unconnected-(U3-PA27-Pad51) -> GND
- U3 pad 52: Net-(U3-~{RESET}) -> GND
- U3 pad 53: Net-(U3-VDDCORE) -> GND
- U3 pad 55: unconnected-(U3-VSW-Pad55) -> GND
- U3 pad 56: VCC -> GND
- U3 pad 57: /SAMD51 ESP32/SWCLK -> GND
- U3 pad 58: /SAMD51 ESP32/SWDIO -> GND
- U3 pad 59: unconnected-(U3-PB30-Pad59) -> GND
- U3 pad 60: unconnected-(U3-PB31-Pad60) -> GND
- U3 pad 61: unconnected-(U3-PB00-Pad61) -> GND
- U3 pad 7: GND -> unconnected-(U3-NC_2-Pad7)
- U3 pad 8: Net-(U3-VDDANA) -> /SAMD51 ESP32/ESP_EN
- U4 pad 1: GND -> +3V8
- U4 pad 3: VCC -> +3V8
- U4 pad 5: unconnected-(U4-IO2-Pad5) -> VCC
- U5 pad 1: +3V8 -> VCC
- U5 pad 2: GND -> Net-(U5-K)
- U5 pad 3: +3V8 -> /SENSOR ARRAY/S0
- U5 pad 4: unconnected-(U5-NC-Pad4) -> GND
- U6 pad 1: VCC -> Net-(U6-A)
- U6 pad 2: Net-(U6-K) -> /SENSOR ARRAY/0_15_LED
- U6 pad 3: /SENSOR ARRAY/S0 -> /SENSOR ARRAY/S15
- U7 pad 1: Net-(U7-A) -> VCC
- U7 pad 2: /SENSOR ARRAY/0_15_LED -> Net-(U7-K)
- U7 pad 3: /SENSOR ARRAY/S15 -> /SENSOR ARRAY/S1
- U8 pad 1: VCC -> Net-(U8-A)
- U8 pad 2: Net-(U8-K) -> /SENSOR ARRAY/1_14_LED
- U8 pad 3: /SENSOR ARRAY/S1 -> /SENSOR ARRAY/S14
- U9 pad 1: Net-(U9-A) -> VCC
- U9 pad 2: /SENSOR ARRAY/1_14_LED -> Net-(U9-K)
- U9 pad 3: /SENSOR ARRAY/S14 -> /SENSOR ARRAY/S2
Other:
- board size 127.2 x 119.8 mm -> 120 x 81.3 mm
- board text added: "MOTOR A"
- board text added: "MOTOR B"

Commit message: Assigned Pins on SAMD51 using Pin Planner and PMODE is hardwired to VCC (PWM mode).
Parts:
- removed C30, C31, C32: 100nF, Capacitor_SMD:C_0402_1005Metric
- removed C33: 100nF/50V, Capacitor_SMD:C_0402_1005Metric
- removed J1, J2: FH34SRJ-8S-0.5SH_50_, SAVITAR:FH34SRJ8S05SH50
- removed MUX1, MUX2: 74HC4051, Package_SO:SOIC-16_3.9x9.9mm_P1.27mm
- removed NMOS1: TBD62083AFNG_Z,EL_, SAVITAR:SOP65P640X155-18N
- removed R37, R39: 47kΩ, Resistor_SMD:R_0402_1005Metric
- removed UNOT1: TEENSY 4.0, SAVITAR:MODULE_DEV-15583
- added Q2: BSS138, Package_TO_SOT_SMD:SOT-23, F.Cu at (153.8, -26.0)
- added Q3: BSS138, Package_TO_SOT_SMD:SOT-23, F.Cu at (153.8, -21.6)
- added Q4: BSS138, Package_TO_SOT_SMD:SOT-23, F.Cu at (158.8, -26.0)
- added Q5: BSS138, Package_TO_SOT_SMD:SOT-23, F.Cu at (158.8, -21.6)
- added Q6: BSS138, Package_TO_SOT_SMD:SOT-23, F.Cu at (163.7, -26.0)
- added Q7: BSS138, Package_TO_SOT_SMD:SOT-23, F.Cu at (163.7, -21.6)
- added Q8: BSS138, Package_TO_SOT_SMD:SOT-23, F.Cu at (168.6, -26.0)
- added Q9: BSS138, Package_TO_SOT_SMD:SOT-23, F.Cu at (168.6, -21.6)
- added R41: 47kΩ, Resistor_SMD:R_0402_1005Metric, F.Cu at (152.8, -18.3)
- added R42: 47kΩ, Resistor_SMD:R_0402_1005Metric, F.Cu at (152.8, -16.3)
- added R43: 47kΩ, Resistor_SMD:R_0402_1005Metric, F.Cu at (152.8, -14.3)
- added R44: 47kΩ, Resistor_SMD:R_0402_1005Metric, F.Cu at (152.8, -12.4)
- added R45: 47kΩ, Resistor_SMD:R_0402_1005Metric, F.Cu at (155.8, -18.3)
- added R46: 47kΩ, Resistor_SMD:R_0402_1005Metric, F.Cu at (155.8, -16.3)
- added R47: 47kΩ, Resistor_SMD:R_0402_1005Metric, F.Cu at (155.8, -14.3)
- added R48: 47kΩ, Resistor_SMD:R_0402_1005Metric, F.Cu at (155.8, -12.4)
- added R49: 47kΩ, Resistor_SMD:R_0402_1005Metric, F.Cu at (158.7, -18.3)
- added R50: 47kΩ, Resistor_SMD:R_0402_1005Metric, F.Cu at (158.7, -16.3)
- added R51: 47kΩ, Resistor_SMD:R_0402_1005Metric, F.Cu at (158.7, -14.3)
- added R52: 47kΩ, Resistor_SMD:R_0402_1005Metric, F.Cu at (158.7, -12.4)
- added R53: 47kΩ, Resistor_SMD:R_0402_1005Metric, F.Cu at (161.6, -18.3)
- added R54: 47kΩ, Resistor_SMD:R_0402_1005Metric, F.Cu at (161.6, -16.3)
- added R55: 47kΩ, Resistor_SMD:R_0402_1005Metric, F.Cu at (161.6, -14.3)
- added R56: 47kΩ, Resistor_SMD:R_0402_1005Metric, F.Cu at (161.6, -12.4)
- FB1: value 50mΩ 2A -> 380mΩ 500mA
- turned U2 to 180 degrees
Connections:
- net /SAMD51 ESP32/MOT_A.PMODE renamed Net-(DRV1-PMODE)
- net /SAMD51 ESP32/MOT_B.PMODE renamed Net-(DRV2-PMODE)
- net /SAMD51 ESP32/SWD1 renamed VCCANA
- DEMUX1 pad 1: /SENSOR ARRAY/S0 -> /SENSOR ARRAY/A0
- DEMUX1 pad 10: /SENSOR ARRAY/I6 -> /SENSOR ARRAY/P6
- DEMUX1 pad 11: /SENSOR ARRAY/I5 -> /SENSOR ARRAY/P5
- DEMUX1 pad 12: /SENSOR ARRAY/I4 -> /SENSOR ARRAY/P4
- DEMUX1 pad 13: /SENSOR ARRAY/I3 -> /SENSOR ARRAY/P3
- DEMUX1 pad 14: /SENSOR ARRAY/I2 -> /SENSOR ARRAY/P2
- DEMUX1 pad 15: /SENSOR ARRAY/I1 -> /SENSOR ARRAY/P1
- DEMUX1 pad 2: /SENSOR ARRAY/S1 -> /SENSOR ARRAY/A1
- DEMUX1 pad 3: /SENSOR ARRAY/S2 -> /SENSOR ARRAY/A2
- DEMUX1 pad 7: /SENSOR ARRAY/I8 -> /SENSOR ARRAY/P8
- DEMUX1 pad 9: /SENSOR ARRAY/I7 -> /SENSOR ARRAY/P7
- DRV1 pad 8: /SAMD51 ESP32/SENSE_IN_A1 -> /SAMD51 ESP32/MOT_A1
- DRV2 pad 8: /SAMD51 ESP32/SENSE_IN_B1 -> /SAMD51 ESP32/MOT_B1
- R21 pad 1: /SAMD51 ESP32/SAMD_TX1 -> /SAMD51 ESP32/ESP_RX
- R22 pad 1: /SAMD51 ESP32/SAMD_RX1 -> /SAMD51 ESP32/ESP_TX
- U2 pad 10: unconnected-(U2-PB07-Pad10) -> /SAMD51 ESP32/SEN_S8
- U2 pad 11: unconnected-(U2-PB08-Pad11) -> /SAMD51 ESP32/SEN_S15
- U2 pad 12: unconnected-(U2-PB09-Pad12) -> /SAMD51 ESP32/SEN_S14
- U2 pad 13: unconnected-(U2-PA04-Pad13) -> /SAMD51 ESP32/SEN_S2
- U2 pad 14: unconnected-(U2-PA05-Pad14) -> /SAMD51 ESP32/SEN_S3
- U2 pad 15: unconnected-(U2-PA06-Pad15) -> /SAMD51 ESP32/SEN_S4
- U2 pad 16: unconnected-(U2-PA07-Pad16) -> /SAMD51 ESP32/SEN_S5
- U2 pad 17: unconnected-(U2-PA08-Pad17) -> /SAMD51 ESP32/SEN_S13
- U2 pad 18: unconnected-(U2-PA09-Pad18) -> /SAMD51 ESP32/SEN_S12
- U2 pad 19: unconnected-(U2-PA10-Pad19) -> /SAMD51 ESP32/SEN_S6
- U2 pad 2: unconnected-(U2-PA01-Pad2) -> /SAMD51 ESP32/SEN_EN
- U2 pad 20: unconnected-(U2-PA11-Pad20) -> /SAMD51 ESP32/SEN_S7
- U2 pad 25: unconnected-(U2-PB12-Pad25) -> /SAMD51 ESP32/SEN_A0
- U2 pad 26: unconnected-(U2-PB13-Pad26) -> /SAMD51 ESP32/SEN_A1
- U2 pad 27: unconnected-(U2-PB14-Pad27) -> /SAMD51 ESP32/SEN_A2
- U2 pad 28: unconnected-(U2-PB15-Pad28) -> /SAMD51 ESP32/STATUS_LED
- U2 pad 29: unconnected-(U2-PA12-Pad29) -> /SAMD51 ESP32/ESP_TX
- U2 pad 3: unconnected-(U2-PA02-Pad3) -> /SAMD51 ESP32/SEN_S0
- U2 pad 30: unconnected-(U2-PA13-Pad30) -> /SAMD51 ESP32/ESP_RX
- U2 pad 35: unconnected-(U2-PA16-Pad35) -> /SAMD51 ESP32/MOT_A.~{SLEEP}
- U2 pad 36: unconnected-(U2-PA17-Pad36) -> /SAMD51 ESP32/MOT_A.~{FAULT}
- U2 pad 37: unconnected-(U2-PA18-Pad37) -> /SAMD51 ESP32/MOT_A.EN/IN1
- U2 pad 38: unconnected-(U2-PA19-Pad38) -> /SAMD51 ESP32/MOT_A.PH/IN2
- U2 pad 4: unconnected-(U2-PA03-Pad4) -> /SAMD51 ESP32/SEN_S1
- U2 pad 43: unconnected-(U2-PA22-Pad43) -> /SAMD51 ESP32/MOT_B.EN/IN1
- U2 pad 44: unconnected-(U2-PA23-Pad44) -> /SAMD51 ESP32/MOT_B.PH/IN2
- U2 pad 5: unconnected-(U2-PB04-Pad5) -> /SAMD51 ESP32/SEN_S11
- U2 pad 59: unconnected-(U2-PB30-Pad59) -> /SAMD51 ESP32/MOT_B.~{SLEEP}
- U2 pad 6: unconnected-(U2-PB05-Pad6) -> /SAMD51 ESP32/SEN_S10
- U2 pad 60: unconnected-(U2-PB31-Pad60) -> /SAMD51 ESP32/MOT_B.~{FAULT}
- U2 pad 61: unconnected-(U2-PB00-Pad61) -> /SAMD51 ESP32/MOT_A.C_STALL
- U2 pad 62: unconnected-(U2-PB01-Pad62) -> /SAMD51 ESP32/MOT_B.C_STALL
- U2 pad 63: unconnected-(U2-PB02-Pad63) -> /SAMD51 ESP32/BAT_LEVEL
- U2 pad 9: unconnected-(U2-PB06-Pad9) -> /SAMD51 ESP32/SEN_S9

Commit message: Updated
Parts:
- moved C18 135.4 mm to (196.7, 212.1), turned to 90 degrees
- moved C20 129.7 mm to (198.4, 212.3), turned to -90 degrees
- moved R23 123.5 mm to (197.7, 205.6), turned to 180 degrees
- moved C7 122.1 mm to (196.4, 177.6), turned to -90 degrees
- moved R24 108.8 mm to (184.4, 201.3)
- moved R20 101.2 mm to (182.2, 199.8)
- moved C8 95.4 mm to (189.9, 169.6)
- moved C10 94.8 mm to (187.9, 184.6)
- moved R13 89.8 mm to (241.9, 167.2)
- moved R14 89.8 mm to (241.9, 169.8)
- moved R18 89.8 mm to (241.9, 179.8)
- moved R19 89.8 mm to (241.9, 182.3)
- moved C9 88.3 mm to (181.4, 180.6), turned to -90 degrees
- moved R17 87.2 mm to (147.6, 211.3)
- moved C11 86.4 mm to (181.4, 173.3), turned to -90 degrees
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Connections:
- net /SAMD51 ESP32/SWD5 renamed /SAMD51 ESP32/RST
- net Net-(D1-A) renamed /SAMD51 ESP32/ANODE1
- net Net-(D2-A) renamed /SAMD51 ESP32/ANODE2
- net Net-(DRV1-PMODE) renamed /SAMD51 ESP32/PMODE_A
- net Net-(DRV1-VCP) renamed /SAMD51 ESP32/VCP_A
- net Net-(DRV2-CPH) renamed /SAMD51 ESP32/CPH_B
- net Net-(DRV2-CPL) renamed /SAMD51 ESP32/CPL_B
- net Net-(DRV2-PMODE) renamed /SAMD51 ESP32/PMODE_B
- net Net-(DRV2-VCP) renamed /SAMD51 ESP32/VCP_B
- net Net-(IC1-FB) renamed /SAMD51 ESP32/FB
- net Net-(U1-I/O1-Pad1) renamed /SAMD51 ESP32/USB_D-
- net Net-(U1-I/O2-Pad3) renamed /SAMD51 ESP32/USB_D+
- net Net-(U3-IO18) renamed /SAMD51 ESP32/IO18
- net Net-(U3-IO19) renamed /SAMD51 ESP32/IO19
- net Net-(U3-IO2) renamed /SAMD51 ESP32/IO2
- net Net-(U3-IO8) renamed /SAMD51 ESP32/IO8
- net Net-(U3-RXD0) renamed /SAMD51 ESP32/RX
- net Net-(U3-TXD0) renamed /SAMD51 ESP32/TX
- net Net-(USBC1-CC1) renamed /SAMD51 ESP32/CC1
- net Net-(USBC1-CC2) renamed /SAMD51 ESP32/CC2
- C4 pad 1: Net-(DRV1-CPH) -> /SAMD51 ESP32/CPL_A
- C4 pad 2: Net-(DRV1-CPL) -> /SAMD51 ESP32/CPL_A
- DRV1 pad 13: Net-(DRV1-CPH) -> /SAMD51 ESP32/CPL_A
- DRV1 pad 14: Net-(DRV1-CPL) -> /SAMD51 ESP32/CPL_A
Other:
- board size 120 x 81.3 mm -> 120 x 82.5 mm
