File: SENSOR_ARRAY.kicad_sch (KiCad schematic)
At the start: 44 parts, among them J2 FH34SRJ-8S-0.5SH_50_, Q1 MMBT3904, U10 QRE1113GR, U11 QRE1113GR, U12 QRE1113GR, U13 QRE1113GR, U14 QRE1113GR, U15 QRE1113GR, U16 QRE1113GR, U17 QRE1113GR, U18 QRE1113GR, U19 QRE1113GR, U20 QRE1113GR, U21 QRE1113GR, U6 QRE1113GR, U7 QRE1113GR, U8 QRE1113GR, U9 QRE1113GR

Commit message: Will add info in a later commit
Parts:
- removed C43, C44, C45: 100nF, Capacitor_SMD:C_0402_1005Metric, symbol Device:C
- removed C46: 100nF/50V, Capacitor_SMD:C_0402_1005Metric, symbol Device:C
- removed J2: FH34SRJ-8S-0.5SH_50_, SAVITAR:FH34SRJ8S05SH50, symbol SAVITAR:FH34SRJ-8S-0.5SH_50_
- removed MUX1, MUX2: 74HC4051, Package_SO:SOIC-16_3.9x9.9mm_P1.27mm, symbol 74xx:74HC4051
- removed NMOS1: TBD62083AFNG_Z,EL_, SAVITAR:SOP65P640X155-18N, symbol SAVITAR:TBD62083AFNG_Z,EL_
- removed R40: 47kΩ, Resistor_SMD:R_0402_1005Metric, symbol Device:R_US
- added FPC1: FPC-05F-22PH20, EasyEDA:FPC-SMD_22P-P0.50_FPC-05F-22PH20, symbol EasyEDA:FPC-05F-22PH20
- added Q2, Q3, Q4, Q5, Q6, Q7, Q8, Q9: BSS138, Package_TO_SOT_SMD:SOT-23, symbol Transistor_FET:BSS138
- added R41, R43, R44, R45, R46, R47, R48, R49, R50, R51, R52, R53, R54, R55, R56: 47kΩ, Resistor_SMD:R_0402_1005Metric, symbol Device:R_US
- renumbered C41 to C28, C42 to C29, R30 to R27, R31 to R28, R32 to R29, R33 to R30, R34 to R31, R35 to R32, R36 to R33, R37 to R34, R38 to R35, R39 to R36, R41 to R38, R43 to R40, U11 to U10, U12 to U11, U13 to U12, U14 to U13, U15 to U14, U16 to U15, U17 to U16, U18 to U17, U19 to U18, U20 to U19, U21 to U20, U6 to U5, U7 to U6, U8 to U7, U9 to U8, U10 to U9
Connections:
- net COUT1 is gone; now on net S15: R42.1
- net 0_15_LED: now also Q9.3 (D)
- net 1_14_LED: now also Q8.3 (D)
- net 2_13_LED: now also Q7.3 (D)
- net 3_12_LED: now also Q6.3 (D)
- net 4_11_LED: now also Q5.3 (D)
- net 5_10_LED: now also Q4.3 (D)
- net 6_9_LED: now also Q3.3 (D)
- net 7_8_LED: now also Q2.3 (D)
- net EN: now also FPC1.22
- net GND: now also FPC1.1, FPC1.23, FPC1.24, Q2.2 (S), Q3.2 (S), Q4.2 (S), Q5.2 (S), Q6.2 (S), Q7.2 (S), Q8.2 (S), Q9.2 (S)
- net S0: now also FPC1.3, R41.1; no longer DEMUX1.1 (A0)
- net S1: now also FPC1.4, R43.1; no longer DEMUX1.2 (A1)
- net S10: now also FPC1.13, R52.1
- net S11: now also FPC1.14, R50.1
- net S12: now also FPC1.15, R48.1
- net S13: now also FPC1.16, R46.1
- net S14: now also FPC1.17, R44.1
- net S15: now also FPC1.18
- net S2: now also FPC1.5, R45.1; no longer DEMUX1.3 (A2)
- net S3: now also FPC1.6, R47.1
- net S4: now also FPC1.7, R49.1
- net S5: now also FPC1.8, R51.1
- net S6: now also FPC1.9, R53.1
- net S7: now also FPC1.10, R55.1
- net S8: now also FPC1.11, R56.1
- net S9: now also FPC1.12, R54.1
- net VCC: now also FPC1.2, R41.2, R43.2, R44.2, R45.2, R46.2, R47.2, R48.2, R49.2, R50.2, R51.2, R52.2, R53.2, R54.2, R55.2, R56.2
- net I1 renamed P1
- net P1: now also Q2.1 (G)
- net I2 renamed P2
- net P2: now also Q3.1 (G)
- net I3 renamed P3
- net P3: now also Q4.1 (G)
- net I4 renamed P4
- net P4: now also Q5.1 (G)
- net I5 renamed P5
- net P5: now also Q6.1 (G)
- net I6 renamed P6
- net P6: now also Q7.1 (G)
- net I7 renamed P7
- net P7: now also Q8.1 (G)
- net I8 renamed P8
- net P8: now also Q9.1 (G)
- new net A0: DEMUX1.1 (A0), FPC1.19
- new net A1: DEMUX1.2 (A1), FPC1.20
- new net A2: DEMUX1.3 (A2), FPC1.21
- no-connect marks 1 -> 0
Other:
- note added: "SELECT ADDR 0 |-> NMOS 0 Triggered -> LED 0 & LED 15 ON -> OFF |-> WAIT TILL STABLE -> READ ADC0 & ADC1"
- note removed: "One for each IC."
- note removed: "READ PAIR"
- note removed: "SELECT ADDR 0 |-> NMOS 0 Triggered -> LED 0 & LED 15 ON -> OFF |-> WAIT TILL STABLE -> READ MUX1 & MUX2"
- moved on the sheet: DEMUX1, Q1, R33, R34, R35, R36, R38, R40, U13, U14, U15, U16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
